File: pcb/battery_protect.kicad_sch (KiCad schematic)
At the start: 139 parts, among them Q18 MMBT5550, Q19 MMBT5550, Q20 MMBT5550, Q21 MMBT5550, Q22 MMBT5550, Q23 MMBT5550, Q24 MMBT5550, Q25 MMBT5550, Q26 MMBT5550, Q27 MMBT5550, Q28 D2PAK-7PIN-IRL40SC228, Q29 D2PAK-7PIN-IRL40SC228, Q30 MMBT5401, Q31 D2PAK-7PIN-IRL40SC228, Q32 D2PAK-7PIN-IRL40SC228, U14 TSSOP28-SH3676010BX/028XY

Commit message: feat: update
Parts:
- B+1: renamed from B+2; VALUE NC -> (none)
- B-1: renamed from B-2; VALUE NC -> (none)
- C1: renamed from C36; VALUE 1uF/25V -> (none)
- C10: renamed from C45; VALUE 0.1uF -> (none)
- C11: renamed from C46; VALUE 1uF/25V -> (none)
- C12: renamed from C47; VALUE 1NF -> (none)
- C13: renamed from C48; VALUE 1uF/25V -> (none)
- C14: renamed from C49; VALUE 1NF -> (none)
- C15: renamed from C50; VALUE 1NF -> (none)
- C16: renamed from C51; VALUE 2.2uF/100V -> (none)
- C17: renamed from C52; VALUE 2.2uF/100V -> (none)
- C18: renamed from C53; VALUE 1NF -> (none)
- C19: renamed from C54; VALUE 1uF/25V -> (none)
- C2: renamed from C37; VALUE 0.1uF -> (none)
- C20: renamed from C55; VALUE 0.1uF/100V -> (none)
- C21: renamed from C56; VALUE 0.1uF/100V -> (none)
- C22: renamed from C57; VALUE 0.1uF/100V -> (none)
- C23: renamed from C58; VALUE 0.1uF/100V -> (none)
- C3: renamed from C38; VALUE 0.1uF -> (none)
- C4: renamed from C39; VALUE 0.1uF -> (none)
- C5: renamed from C40; VALUE 0.1uF -> (none)
- C6: renamed from C41; VALUE 0.1uF -> (none)
- C7: renamed from C42; VALUE 0.1uF -> (none)
- C8: renamed from C43; VALUE 0.1uF -> (none)
- C9: renamed from C44; VALUE 0.1uF -> (none)
- D1: renamed from D23; VALUE LED RED -> (none)
- D10: renamed from D32; VALUE LED RED -> (none)
- D11: renamed from D33; VALUE IN4148W -> (none)
- D12: renamed from D34; VALUE IN4148W -> (none)
- D13: renamed from D35; VALUE BAV21W -> (none)
- D14: renamed from D36; VALUE SMBJ64A SMB -> (none)
- D15: renamed from D37; VALUE SOD-323 BZT52C15 -> (none)
- D16: renamed from D38; VALUE IN4148W -> (none)
- D17: renamed from D39; VALUE SOD-323 BZT52C15 -> (none)
- D18: renamed from D40; VALUE RS3M SMC -> (none)
- D19: renamed from D41; VALUE BAV21W -> (none)
- D2: renamed from D24; VALUE LED RED -> (none)
- D3: renamed from D25; VALUE LED RED -> (none)
- D4: renamed from D26; VALUE LED RED -> (none)
- D5: renamed from D27; VALUE LED RED -> (none)
- D6: renamed from D28; VALUE LED RED -> (none)
- D7: renamed from D29; VALUE LED RED -> (none)
- D8: renamed from D30; VALUE LED RED -> (none)
- D9: renamed from D31; VALUE LED RED -> (none)
- NTC1: renamed from NTC4; value NTC 10K±1% -> 10K; VALUE 10K -> (none)
- NTC2: renamed from NTC5; value NTC 10K±1% -> 10K; VALUE 10K -> (none)
- NTC3: renamed from NTC6; value NTC 10K±1% -> 10K; VALUE 10K -> (none)
- Q1: renamed from Q18; VALUE MMBT5550 -> (none)
- Q10: renamed from Q27; VALUE MMBT5550 -> (none)
- Q11: renamed from Q28; VALUE D2PAK-7PIN-IRL40SC228 -> (none)
- Q12: renamed from Q29; VALUE D2PAK-7PIN-IRL40SC228 -> (none)
- Q13: renamed from Q30; VALUE MMBT5401 -> (none)
- Q14: renamed from Q31; VALUE D2PAK-7PIN-IRL40SC228 -> (none)
- Q15: renamed from Q32; VALUE D2PAK-7PIN-IRL40SC228 -> (none)
- Q2: renamed from Q19; VALUE MMBT5550 -> (none)
- Q3: renamed from Q20; VALUE MMBT5550 -> (none)
- Q4: renamed from Q21; VALUE MMBT5550 -> (none)
- Q5: renamed from Q22; VALUE MMBT5550 -> (none)
- Q6: renamed from Q23; VALUE MMBT5550 -> (none)
- Q7: renamed from Q24; VALUE MMBT5550 -> (none)
- Q8: renamed from Q25; VALUE MMBT5550 -> (none)
- Q9: renamed from Q26; VALUE MMBT5550 -> (none)
- R1: renamed from R78; VALUE 47R 1206 -> (none)
- R10: renamed from R87; VALUE 47R 2512 -> (none)
- R11: renamed from R88; VALUE 47R 2512 -> (none)
- R12: renamed from R89; VALUE 2.7K -> (none)
- R13: renamed from R90; VALUE 2.7K -> (none)
- R14: renamed from R91; VALUE 2.7K -> (none)
- R15: renamed from R92; VALUE 2.7K -> (none)
- R16: renamed from R93; VALUE 2.7K -> (none)
- R17: renamed from R94; VALUE 2.7K -> (none)
- R18: renamed from R95; VALUE 2.7K -> (none)
- R19: renamed from R96; VALUE 2.7K -> (none)
- R2: renamed from R79; VALUE 47R 2512 -> (none)
- R20: renamed from R97; VALUE 2.7K -> (none)
- R21: renamed from R98; VALUE 2.7K -> (none)
- R22: renamed from R99; VALUE 510R -> (none)
- R23: renamed from R100; VALUE 510R -> (none)
- R24: renamed from R101; VALUE 510R -> (none)
- R25: renamed from R102; VALUE 510R -> (none)
- R26: renamed from R103; VALUE 510R -> (none)
- R27: renamed from R104; VALUE 510R -> (none)
- R28: renamed from R105; VALUE 510R -> (none)
- R29: renamed from R106; VALUE 510R -> (none)
- R3: renamed from R80; VALUE 47R 2512 -> (none)
- R30: renamed from R107; VALUE 510R -> (none)
- R31: renamed from R108; VALUE 510R -> (none)
- R32: renamed from R109; VALUE 510R -> (none)
- R33: renamed from R110; VALUE 510R -> (none)
- R34: renamed from R111; VALUE 510R -> (none)
- R35: renamed from R112; VALUE 510R -> (none)
- R36: renamed from R113; VALUE 510R -> (none)
- R37: renamed from R114; VALUE 510R -> (none)
- R38: renamed from R115; VALUE 510R -> (none)
- R39: renamed from R116; VALUE 510R -> (none)
- R4: renamed from R81; VALUE 47R 2512 -> (none)
- R40: renamed from R117; VALUE 510R -> (none)
- R41: renamed from R118; VALUE 510R -> (none)
- R42: renamed from R119; VALUE 510R -> (none)
- R43: renamed from R120; VALUE 10R 0805 -> (none)
- R44: renamed from R121; VALUE 0.005R 2512 -> (none)
- R45: renamed from R122; VALUE 0.005R 2512 -> (none)
- R46: renamed from R123; VALUE 0.005R 2512 -> (none)
- R47: renamed from R124; VALUE 0.005R 2512 -> (none)
- R48: renamed from R125; VALUE 0.005R 2512 -> (none)
- R49: renamed from R126; VALUE 10R 0805 -> (none)
- R5: renamed from R82; VALUE 47R 2512 -> (none)
- R50: renamed from R127; VALUE NC -> (none)
- R51: renamed from R128; VALUE 1K 0805 -> (none)
- R52: renamed from R129; VALUE 1K 0805 -> (none)
- R53: renamed from R130; VALUE 3M -> (none)
- R54: renamed from R131; VALUE 1M -> (none)
- R55: renamed from R132; VALUE 1K -> (none)
- R56: renamed from R133; VALUE 1K -> (none)
- R57: renamed from R134; VALUE 1K -> (none)
- R58: renamed from R135; VALUE 10K -> (none)
- R59: renamed from R136; VALUE 10K -> (none)
- R6: renamed from R83; VALUE 47R 2512 -> (none)
- R60: renamed from R137; VALUE 10M -> (none)
- R61: renamed from R138; VALUE 47R 1206 -> (none)
- R62: renamed from R139; VALUE 47R 1206 -> (none)
- R63: renamed from R140; VALUE 1M -> (none)
- R64: renamed from R141; VALUE 3M -> (none)
- R65: renamed from R142; VALUE 47R 1206 -> (none)
- R66: renamed from R143; VALUE 47R 1206 -> (none)
- R67: renamed from R144; VALUE 1M -> (none)
- R68: renamed from R145; VALUE 100R -> (none)
- R69: renamed from R146; VALUE 100R -> (none)
- R7: renamed from R84; VALUE 47R 2512 -> (none)
- R8: renamed from R85; VALUE 47R 2512 -> (none)
- R9: renamed from R86; VALUE 47R 2512 -> (none)
- U2: renamed from U14; value TSSOP28-SH3676010BX/028XY -> TSSOP28-SH3676010B; VALUE TSSOP28-SH3676010B -> (none)
- renumbered J2 to J1, LED2 to LED1, R147 to R70, U13 to U1, U15 to U3, U16 to U4, U17 to U5
