File: pcb/main_ctrl.kicad_sch (KiCad schematic)
At the start: 43 parts, among them Q3 S8050, Q4 S8050, U4 CP2102N-A02-GQFN28

Commit message: feat: update
Parts:
- renumbered C14 to C45, C15 to C46, C9 to C47, C12 to C48, C13 to C49, C10 to C50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
Changed lines of the file:
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@@
 (kicad_sch
-	(version 20231120)
+	(version 20250227)
 	(generator "eeschema")
-	(generator_version "8.0")
+	(generator_version "9.99")
 	(paper "A4")
