File: pcb/skateboard.kicad_pcb (KiCad board)
At the start: 2 copper layers, 0 parts

Commit message: feat: update
Parts:
- added C24: 4.7uf/50v, Capacitor_SMD:C_1206_3216Metric, F.Cu at (151.2, 84.1)
- added C25: 4.7uf/50v, Capacitor_SMD:C_1206_3216Metric, F.Cu at (151.2, 87.4)
- added C26: 4.7uf/50v, Capacitor_SMD:C_1206_3216Metric, F.Cu at (151.2, 90.8)
- added C27: 100nf/50v, Capacitor_SMD:C_0603_1608Metric, F.Cu at (125.8, 83.7)
- added C28: 10uf/50v, Capacitor_SMD:C_1210_3225Metric, F.Cu at (137.5, 104.6)
- added C29: 100nf/50v, Capacitor_SMD:C_0603_1608Metric, F.Cu at (125.8, 86.2)
- added C30: 10uf/50v, Capacitor_SMD:C_1210_3225Metric, F.Cu at (137.5, 108.9)
- added C31: 68nF, Capacitor_SMD:C_0603_1608Metric, F.Cu at (125.8, 88.7)
- added C32: 47nF, Capacitor_SMD:C_0603_1608Metric, F.Cu at (125.8, 91.2)
- added C33: 47nF, Capacitor_SMD:C_0603_1608Metric, F.Cu at (125.8, 93.7)
- added C34: 100nF/16v, Capacitor_SMD:C_0603_1608Metric, F.Cu at (125.8, 96.2)
- added C35: 100nF/16v, Capacitor_SMD:C_0603_1608Metric, F.Cu at (125.8, 98.7)
- added C36: 100nF/16v, Capacitor_SMD:C_0603_1608Metric, F.Cu at (125.8, 101.2)
- added C37: 10uF/35v, Capacitor_SMD:C_1210_3225Metric, F.Cu at (137.5, 113.1)
- added C38: 10uF/35v, Capacitor_SMD:C_1210_3225Metric, F.Cu at (137.5, 117.4)
- added C39: 10uF/16v, Capacitor_SMD:C_1210_3225Metric, F.Cu at (137.5, 121.6)
- added C40: 10uF/16v, Capacitor_SMD:C_1210_3225Metric, F.Cu at (137.5, 125.9)
- added C41: 10uF/10v, Capacitor_SMD:C_0603_1608Metric, F.Cu at (129.8, 83.7)
- added C42: 10uF/10v, Capacitor_SMD:C_0603_1608Metric, F.Cu at (129.8, 86.2)
- added C43: 10uF, Capacitor_SMD:C_0603_1608Metric, F.Cu at (129.8, 88.7)
- added C44: 0.1uF, Capacitor_SMD:C_0603_1608Metric, F.Cu at (129.8, 91.2)
- added C47: 1uF(105), Capacitor_SMD:C_0402_1005Metric, F.Cu at (170.4, 83.4)
- added C48: 10uF, Capacitor_SMD:C_1206_3216Metric, F.Cu at (161.9, 84.1)
- added C49: 1uF(105), Capacitor_SMD:C_0402_1005Metric, F.Cu at (170.4, 85.4)
- added C50: 1uF(105), Capacitor_SMD:C_0402_1005Metric, F.Cu at (170.4, 87.3)
- added C51: 1uF(105), Capacitor_SMD:C_0402_1005Metric, F.Cu at (170.4, 89.3)
- added C52: 10uF, Capacitor_SMD:C_1206_3216Metric, F.Cu at (161.9, 87.4)
- added C53: 10uF, Capacitor_SMD:C_1206_3216Metric, F.Cu at (161.9, 90.8)
- added D20: B560C, Diode_SMD:D_SMC, F.Cu at (129.3, 106.4)
- added D21: B560C, Diode_SMD:D_SMC, F.Cu at (129.3, 114.1)
- added D22: B560C, Diode_SMD:D_SMC, F.Cu at (129.3, 121.9)
- added D27: MM1Z20V, lceda:SOD-123_L2.8-W1.8-LS3.7-RD, F.Cu at (164.2, 93.9)
- added J2: sig_in, Connector_PinHeader_2.54mm:PinHeader_1x02_P2.54mm_Vertical, F.Cu at (142.2, 96.4)
- added J3: sig_out, Connector_PinHeader_2.54mm:PinHeader_1x02_P2.54mm_Vertical, F.Cu at (146.8, 96.4)
- added J4: Conn_02x02_Counter_Clockwise, Connector_PinHeader_2.54mm:PinHeader_2x02_P2.54mm_Vertical, F.Cu at (142.7, 124.8)
- added L1: 22uH, Inductor_SMD:L_TDK_SLF12565, F.Cu at (116.2, 89.7)
- added L2: 47uH, Inductor_SMD:L_TDK_SLF12565, F.Cu at (116.2, 104.1)
- added L3: 22uH, Inductor_SMD:L_TDK_SLF12565, F.Cu at (116.2, 118.4)
- added Q16: S8050, lceda:SOT-23-3_L2.9-W1.3-P1.90-LS2.4-BR, F.Cu at (166.8, 84.5)
- added Q17: S8050, lceda:SOT-23-3_L2.9-W1.3-P1.90-LS2.4-BR, F.Cu at (166.8, 88.7)
- added R100: 0, Resistor_SMD:R_0201_0603Metric, F.Cu at (160.3, 98.6)
- added R101: 10K, lceda:R0402, F.Cu at (157.5, 96.4)
- added R102: 10K, lceda:R0402, F.Cu at (157.5, 98.5)
- added R71: 1.3k, Resistor_SMD:R_0603_1608Metric, F.Cu at (129.8, 93.7)
- added R72: 1.3k, Resistor_SMD:R_0603_1608Metric, F.Cu at (129.8, 96.2)
- added R73: 100k, Resistor_SMD:R_0603_1608Metric, F.Cu at (129.8, 98.7)
- added R74: 62k, Resistor_SMD:R_0603_1608Metric, F.Cu at (129.8, 101.2)
- added R75: 62k, Resistor_SMD:R_0603_1608Metric, F.Cu at (133.8, 83.7)
- added R76: 300k, Resistor_SMD:R_0603_1608Metric, F.Cu at (133.8, 86.2)
- added R77: 10k, Resistor_SMD:R_0603_1608Metric, F.Cu at (133.8, 88.7)
- added R78: 10k, Resistor_SMD:R_0603_1608Metric, F.Cu at (133.8, 91.2)
- added R79: 56k, Resistor_SMD:R_0603_1608Metric, F.Cu at (133.8, 93.7)
- added R80: 680, Resistor_SMD:R_0603_1608Metric, F.Cu at (133.8, 96.2)
- added R81: 10k, Resistor_SMD:R_0603_1608Metric, F.Cu at (133.8, 98.7)
- added R82: 33k, Resistor_SMD:R_0603_1608Metric, F.Cu at (133.8, 101.2)
- added R83: 1k, Resistor_SMD:R_0603_1608Metric, F.Cu at (137.8, 83.7)
- added R84: 10k, Resistor_SMD:R_0603_1608Metric, F.Cu at (137.8, 86.2)
- added R85: 120, Resistor_SMD:R_0603_1608Metric, F.Cu at (137.8, 88.7)
- added R86: 100, Resistor_SMD:R_0603_1608Metric, F.Cu at (137.8, 91.2)
- added R87: 100, Resistor_SMD:R_0603_1608Metric, F.Cu at (137.8, 93.7)
- added R88: 5K1, lceda:R0402, F.Cu at (157.5, 83.5)
- added R89: 5K1, lceda:R0402, F.Cu at (157.5, 85.6)
- added R92: 10k, lceda:C0402, F.Cu at (168.6, 93.5)
- added R93: 22.1K, lceda:R0402, F.Cu at (157.5, 87.8)
- added R94: 47.5K, lceda:R0402, F.Cu at (157.5, 89.9)
- added R95: 1K, lceda:R0402, F.Cu at (157.5, 92.1)
- added R96: 10K(NC), lceda:R0402, F.Cu at (157.5, 94.2)
- added R97: 0, Resistor_SMD:R_0201_0603Metric, F.Cu at (160.3, 93.3)
- added R98: 0, Resistor_SMD:R_0201_0603Metric, F.Cu at (160.3, 95.1)
- added R99: 0, Resistor_SMD:R_0201_0603Metric, F.Cu at (160.3, 96.8)
- added RN1: 1k, lceda:RES-ARRAY-SMD_0603-8P-L3.2-W1.6-BL, F.Cu at (164.0, 97.4)
- added SW1: SW_SPST, Button_Switch_SMD:SW_DIP_SPSTx01_Slide_Copal_CHS-01A_W5.08mm_P1.27mm_JPin, F.Cu at (112.7, 127.5)
- added U10: SIT1042AQT/3, Package_DFN_QFN:DFN-8-1EP_3x3mm_P0.65mm_EP1.5x2.25mm, F.Cu at (150.6, 124.8)
- added U2: TSSOP28-SH3676010B, lceda:IC-TSSOP-28, F.Cu at (160.0, 107.0)
- added U6: LMR16030SDDAR, Package_SO:TI_SO-PowerPAD-8_ThermalVias, F.Cu at (144.6, 105.9)
- added U7: LMR16030SDDAR, Package_SO:TI_SO-PowerPAD-8_ThermalVias, F.Cu at (144.6, 112.5)
- added U8: LMR16030SDDAR, Package_SO:TI_SO-PowerPAD-8_ThermalVias, F.Cu at (144.6, 119.2)
- added U9: HX711, Package_SO:SOP-16_3.9x9.9mm_P1.27mm, F.Cu at (144.1, 88.3)
