File: pcb/skateboard.kicad_pcb (KiCad board)
At the start: 2 copper layers, 78 parts, among them J2 sig_in, J3 sig_out, J4 Conn_02x02_Counter_Clockwise, Q16 S8050, Q17 S8050, SW1 SW_SPST, U10 SIT1042AQT/3, U2 TSSOP28-SH3676010B, U6 LMR16030SDDAR, U7 LMR16030SDDAR, U8 LMR16030SDDAR, U9 HX711

Commit message: feat: update
Parts:
- removed D20, D21, D22: B560C, Diode_SMD:D_SMC
- removed D27: MM1Z20V, lceda:SOD-123_L2.8-W1.8-LS3.7-RD
- removed Q16, Q17: S8050, lceda:SOT-23-3_L2.9-W1.3-P1.90-LS2.4-BR
- removed R100, R97, R98, R99: 0, Resistor_SMD:R_0201_0603Metric
- removed R101, R102: 10K, lceda:R0402
- removed R71, R72: 1.3k, Resistor_SMD:R_0603_1608Metric
- removed R73: 100k, Resistor_SMD:R_0603_1608Metric
- removed R74, R75: 62k, Resistor_SMD:R_0603_1608Metric
- removed R76: 300k, Resistor_SMD:R_0603_1608Metric
- removed R77, R78, R81, R84: 10k, Resistor_SMD:R_0603_1608Metric
- removed R79: 56k, Resistor_SMD:R_0603_1608Metric
- removed R80: 680, Resistor_SMD:R_0603_1608Metric
- removed R82: 33k, Resistor_SMD:R_0603_1608Metric
- removed R83: 1k, Resistor_SMD:R_0603_1608Metric
- removed R85: 120, Resistor_SMD:R_0603_1608Metric
- removed R86, R87: 100, Resistor_SMD:R_0603_1608Metric
- removed R88, R89: 5K1, lceda:R0402
- removed R92: 10k, lceda:C0402
- removed R93: 22.1K, lceda:R0402
- removed R94: 47.5K, lceda:R0402
- removed R95: 1K, lceda:R0402
- removed R96: 10K(NC), lceda:R0402
- removed RN1: 1k, lceda:RES-ARRAY-SMD_0603-8P-L3.2-W1.6-BL
- added 3.3V2: LED, LED_SMD:LED_0603_1608Metric, F.Cu at (34.4, 74.0)
- added 3.3V2: LED, LED_SMD:LED_0603_1608Metric, F.Cu at (171.0, 84.5)
- added 3.3V4: LED, LED_SMD:LED_0603_1608Metric, F.Cu at (118.1, 144.3)
- added 3.3V4: LED, LED_SMD:LED_0603_1608Metric, F.Cu at (28.3, 74.0)
- added 42V2: LED, LED_SMD:LED_0603_1608Metric, F.Cu at (171.0, 87.1)
- added 42V2: LED, LED_SMD:LED_0603_1608Metric, F.Cu at (34.4, 76.6)
- added 42V4: LED, LED_SMD:LED_0603_1608Metric, F.Cu at (118.1, 146.9)
- added C1: 10uF, Capacitor_SMD:C_0603_1608Metric, F.Cu at (187.5, 95.7)
- added C10: 10uf/50v, Capacitor_SMD:C_1210_3225Metric, F.Cu at (44.3, 33.4)
- added C11: 68nF, Capacitor_SMD:C_0603_1608Metric, F.Cu at (60.1, 33.3)
- added C12: 100nF/16v, Capacitor_SMD:C_0603_1608Metric, F.Cu at (60.1, 35.8)
- added C13: 100nF/16v, Capacitor_SMD:C_0603_1608Metric, F.Cu at (60.1, 38.3)
- added C14: 10uF/16v, Capacitor_SMD:C_1210_3225Metric, F.Cu at (44.3, 37.7)
- added C15: 10uF/16v, Capacitor_SMD:C_1210_3225Metric, F.Cu at (44.3, 41.9)
- added C16: 10uF/35v, Capacitor_SMD:C_1210_3225Metric, F.Cu at (44.3, 46.2)
- added C17: 10uF/35v, Capacitor_SMD:C_1210_3225Metric, F.Cu at (44.3, 50.4)
- added C18: 47nF, Capacitor_SMD:C_0603_1608Metric, F.Cu at (60.1, 40.9)
- added C19: 100nF/16v, Capacitor_SMD:C_0603_1608Metric, F.Cu at (60.1, 43.4)
- added C2: 100nF, Capacitor_SMD:C_0603_1608Metric, F.Cu at (187.5, 98.2)
- added C20: 4.7uf/50v, Capacitor_SMD:C_1206_3216Metric, F.Cu at (44.3, 54.2)
- added C21: 4.7uf/50v, Capacitor_SMD:C_1206_3216Metric, F.Cu at (44.3, 57.6)
- added C22: 10uF/10v, Capacitor_SMD:C_0603_1608Metric, F.Cu at (64.1, 28.3)
- added C23: 10uF/10v, Capacitor_SMD:C_0603_1608Metric, F.Cu at (64.1, 30.8)
- added C3: 100nf, Capacitor_SMD:C_0603_1608Metric, F.Cu at (107.3, 85.9)
- added C4: 10uF, Capacitor_SMD:C_0603_1608Metric, F.Cu at (187.5, 100.7)
- added C45: 1uF, Capacitor_SMD:C_0603_1608Metric, F.Cu at (107.3, 93.4)
- added C46: 100nF, Capacitor_SMD:C_0603_1608Metric, F.Cu at (123.8, 105.9)
- added C5: 100nF, Capacitor_SMD:C_0603_1608Metric, F.Cu at (187.5, 103.2)
- added C54: 20pF, Capacitor_SMD:C_0603_1608Metric, F.Cu at (123.8, 121.0)
- added C55: 1nF, Capacitor_SMD:C_0603_1608Metric, F.Cu at (127.9, 103.4)
- added C56: 100nF, Capacitor_SMD:C_0603_1608Metric, F.Cu at (127.9, 105.9)
- added C57: 100nF, Capacitor_SMD:C_0603_1608Metric, F.Cu at (127.9, 108.4)
- added C58: 20pF, Capacitor_SMD:C_0603_1608Metric, F.Cu at (127.9, 110.9)
- added C59: 0.1nF, Capacitor_SMD:C_0603_1608Metric, F.Cu at (127.9, 113.4)
- added C60: 0.1nF, Capacitor_SMD:C_0603_1608Metric, F.Cu at (127.9, 115.9)
- added C7: 10uf/50v, Capacitor_SMD:C_1210_3225Metric, F.Cu at (44.3, 29.2)
- added C8: 100nf/50v, Capacitor_SMD:C_0603_1608Metric, F.Cu at (60.1, 28.3)
- added C9: 47nF, Capacitor_SMD:C_0603_1608Metric, F.Cu at (60.1, 30.8)
- added D1: ESD9B5.0ST5G, Diode_SMD:D_SOD-923, F.Cu at (135.2, 95.1)
- added D10: LED, LED_SMD:LED_0603_1608Metric, F.Cu at (131.8, 93.7)
- added D11: B560C, Diode_SMD:D_SMC, F.Cu at (52.6, 30.9)
- added D12: B560C, Diode_SMD:D_SMC, F.Cu at (52.6, 38.7)
- added D13: LED, LED_SMD:LED_0603_1608Metric, F.Cu at (43.6, 63.9)
- added D14: LED, LED_SMD:LED_0603_1608Metric, F.Cu at (43.6, 66.5)
- added D15: SMAJ13CA, Diode_SMD:D_SMA, F.Cu at (235.0, 61.9)
- added D16: B560C, Diode_SMD:D_SMC, F.Cu at (52.6, 46.4)
- added D17: LED, LED_SMD:LED_0603_1608Metric, F.Cu at (43.6, 69.1)
- added D19: LED, LED_SMD:LED_0603_1608Metric, F.Cu at (28.3, 76.6)
- added D2: ESD9B5.0ST5G, Diode_SMD:D_SOD-923, F.Cu at (135.2, 97.1)
- added D3: ESD9B5.0ST5G, Diode_SMD:D_SOD-923, F.Cu at (135.2, 99.0)
- added D4: MBR120VLSFT1G, Diode_SMD:D_SMC, F.Cu at (95.0, 88.5)
- added D5: MBR120VLSFT1G, Diode_SMD:D_SMC, F.Cu at (95.0, 96.3)
- added D6: USB, LED_SMD:LED_0603_1608Metric, F.Cu at (131.8, 85.9)
- added D7: 3.3v, LED_SMD:LED_0603_1608Metric, F.Cu at (131.8, 88.5)
- added D8: SMAJ13CA, Diode_SMD:D_SMA, F.Cu at (235.0, 57.4)
- added D9: LED, LED_SMD:LED_0603_1608Metric, F.Cu at (131.8, 91.1)
- added J1: RC555, Connector_PinHeader_2.54mm:PinHeader_1x08_P2.54mm_Vertical, F.Cu at (243.4, 57.4)
- added J1: sig_in, Connector_PinHeader_2.54mm:PinHeader_1x02_P2.54mm_Vertical, F.Cu at (191.8, 108.4)
- added J10: PH_2.0, Connector_JST:JST_PH_B5B-PH-SM4-TB_1x05-1MP_P2.00mm_Vertical, F.Cu at (97.8, 144.5)
- added J11: adc_sensor2, TerminalBlock:TerminalBlock_MaiXu_MX126-5.0-04P_1x04_P5.00mm, F.Cu at (212.4, 70.2)
- added J12: adc_sensor1, TerminalBlock:TerminalBlock_MaiXu_MX126-5.0-04P_1x04_P5.00mm, F.Cu at (212.4, 80.3)
- added J5: UART, Connector_PinHeader_2.54mm:PinHeader_1x04_P2.54mm_Vertical, F.Cu at (115.7, 87.0)
- added J6: TB_MOTOR, Connector_AMASS:AMASS_MR30PW-M_1x03_P3.50mm_Horizontal, F.Cu at (165.4, 80.7)
- added J7: PH_2.0, Connector_JST:JST_PH_B5B-PH-SM4-TB_1x05-1MP_P2.00mm_Vertical, F.Cu at (150.7, 84.7)
- added J8: sig_in, Connector_PinHeader_2.54mm:PinHeader_1x02_P2.54mm_Vertical, F.Cu at (196.5, 108.4)
- added J8: power, Connector_AMASS:AMASS_XT60PW-M_1x02_P7.20mm_Horizontal, F.Cu at (52.3, 67.7)
- added J9: TB_MOTOR, Connector_AMASS:AMASS_MR30PW-M_1x03_P3.50mm_Horizontal, F.Cu at (112.5, 140.5)
- added Q1: AO3401A, Package_TO_SOT_SMD:SOT-23, F.Cu at (102.9, 87.0)
- added Q2: SS8050, Package_TO_SOT_SMD:SOT-23, F.Cu at (102.9, 91.7)
- added Q3: SS8050, Package_TO_SOT_SMD:SOT-23, F.Cu at (102.9, 96.3)
- added Q4: BTN8982TA, Package_TO_SOT_SMD:TO-263-7_TabPin8, F.Cu at (153.2, 48.6)
- added Q5: BTN8982TA, Package_TO_SOT_SMD:TO-263-7_TabPin8, F.Cu at (153.2, 60.9)
- added Q6: BTN8982TA, Package_TO_SOT_SMD:TO-263-7_TabPin8, F.Cu at (153.2, 73.3)
- added Q7: BTN8982TA, Package_TO_SOT_SMD:TO-263-7_TabPin8, F.Cu at (100.3, 108.3)
- added Q8: BTN8982TA, Package_TO_SOT_SMD:TO-263-7_TabPin8, F.Cu at (100.3, 120.7)
- added Q9: BTN8982TA, Package_TO_SOT_SMD:TO-263-7_TabPin8, F.Cu at (100.3, 133.0)
- added R1: 100, Resistor_SMD:R_0603_1608Metric, F.Cu at (187.5, 105.7)
- added R10: 1.3k, Resistor_SMD:R_0603_1608Metric, F.Cu at (64.1, 35.8)
- added R11: 62k, Resistor_SMD:R_0603_1608Metric, F.Cu at (64.1, 38.3)
- added R12: 100k, Resistor_SMD:R_0603_1608Metric, F.Cu at (64.1, 40.9)
- added R13: 56k, Resistor_SMD:R_0603_1608Metric, F.Cu at (64.1, 43.4)
- added R14: 680, Resistor_SMD:R_0603_1608Metric, F.Cu at (68.1, 28.3)
- added R15: 10k, Resistor_SMD:R_0603_1608Metric, F.Cu at (68.1, 30.8)
- added R16: 300k, Resistor_SMD:R_0603_1608Metric, F.Cu at (68.1, 33.3)
- added R17: 10k, Resistor_SMD:R_0603_1608Metric, F.Cu at (68.1, 35.8)
- added R18: 10k, Resistor_SMD:R_0603_1608Metric, F.Cu at (68.1, 38.3)
- added R19: 10k, Resistor_SMD:R_0603_1608Metric, F.Cu at (68.1, 40.9)
- added R2: 100, Resistor_SMD:R_0603_1608Metric, F.Cu at (187.5, 108.2)
- added R20: 10k, Resistor_SMD:R_0603_1608Metric, F.Cu at (68.1, 43.4)
- added R21: 1.3k, Resistor_SMD:R_0603_1608Metric, F.Cu at (72.1, 28.3)
- added R22: 62k, Resistor_SMD:R_0603_1608Metric, F.Cu at (72.1, 30.8)
- added R23: 10k, Resistor_SMD:R_0603_1608Metric, F.Cu at (72.1, 33.3)
- added R24: 33k, Resistor_SMD:R_0603_1608Metric, F.Cu at (72.1, 35.8)
- added R25: 1k, Resistor_SMD:R_0603_1608Metric, F.Cu at (72.1, 38.3)
- added R26: 10k, Resistor_SMD:R_0603_1608Metric, F.Cu at (72.1, 40.9)
- added R27: 10k, Resistor_SMD:R_0603_1608Metric, F.Cu at (180.8, 58.7)
- added R28: 1k, Resistor_SMD:R_0603_1608Metric, F.Cu at (180.8, 61.2)
- added R29: 10k, Resistor_SMD:R_0603_1608Metric, F.Cu at (184.8, 43.6)
- added R3: 120, Resistor_SMD:R_0603_1608Metric, F.Cu at (187.5, 110.8)
- added R30: 0.51k, Resistor_SMD:R_0603_1608Metric, F.Cu at (184.8, 46.1)
- added R31: 10k, Resistor_SMD:R_0603_1608Metric, F.Cu at (184.8, 48.7)
- added R32: 1k, Resistor_SMD:R_0603_1608Metric, F.Cu at (184.8, 51.2)
- added R33: 3.3k, Resistor_SMD:R_0603_1608Metric, F.Cu at (184.8, 53.7)
- added R34: 10k, Resistor_SMD:R_0603_1608Metric, F.Cu at (184.8, 56.2)
- added R35: 10k, Resistor_SMD:R_0603_1608Metric, F.Cu at (184.8, 58.7)
- added R36: 0.51k, Resistor_SMD:R_0603_1608Metric, F.Cu at (184.8, 61.2)
- added R37: 1k, Resistor_SMD:R_0603_1608Metric, F.Cu at (188.8, 43.6)
- added R38: 3.3k, Resistor_SMD:R_0603_1608Metric, F.Cu at (188.8, 46.1)
- added R39: 10k, Resistor_SMD:R_0603_1608Metric, F.Cu at (188.8, 48.7)
- added R4: 5K1, Resistor_SMD:R_0603_1608Metric, F.Cu at (107.3, 95.9)
- added R40: 1k, Resistor_SMD:R_0603_1608Metric, F.Cu at (188.8, 51.2)
- added R41: 10k, Resistor_SMD:R_0603_1608Metric, F.Cu at (188.8, 53.7)
- added R42: 0.51k, Resistor_SMD:R_0603_1608Metric, F.Cu at (188.8, 56.2)
- added R43: 3.3k, Resistor_SMD:R_0603_1608Metric, F.Cu at (188.8, 58.7)
- added R44: 0.001, Resistor_SMD:R_2512_6332Metric, F.Cu at (186.7, 68.9)
- added R45: 0.001, Resistor_SMD:R_2512_6332Metric, F.Cu at (186.7, 73.8)
- added R46: 100, Resistor_SMD:R_0603_1608Metric, F.Cu at (187.5, 113.3)
- added R47: 100, Resistor_SMD:R_0603_1608Metric, F.Cu at (187.5, 115.8)
- added R48: 10k, Resistor_SMD:R_0603_1608Metric, F.Cu at (127.9, 118.5)
- added R49: 1k, Resistor_SMD:R_0603_1608Metric, F.Cu at (127.9, 121.0)
- added R5: 5K1, Resistor_SMD:R_0603_1608Metric, F.Cu at (111.4, 85.9)
- added R50: 10k, Resistor_SMD:R_0603_1608Metric, F.Cu at (131.9, 103.4)
- added R51: 0.51k, Resistor_SMD:R_0603_1608Metric, F.Cu at (131.9, 105.9)
- added R52: 10k, Resistor_SMD:R_0603_1608Metric, F.Cu at (131.9, 108.4)
- added R53: 1k, Resistor_SMD:R_0603_1608Metric, F.Cu at (131.9, 110.9)
- added R54: 3.3k, Resistor_SMD:R_0603_1608Metric, F.Cu at (131.9, 113.4)
- added R55: 10k, Resistor_SMD:R_0603_1608Metric, F.Cu at (131.9, 115.9)
- added R56: 10k, Resistor_SMD:R_0603_1608Metric, F.Cu at (131.9, 118.5)
- added R57: 0.51k, Resistor_SMD:R_0603_1608Metric, F.Cu at (131.9, 121.0)
- added R58: 1k, Resistor_SMD:R_0603_1608Metric, F.Cu at (135.9, 103.4)
- added R59: 3.3k, Resistor_SMD:R_0603_1608Metric, F.Cu at (135.9, 105.9)
- added R6: 10K, Resistor_SMD:R_0603_1608Metric, F.Cu at (111.4, 88.4)
- added R60: 10k, Resistor_SMD:R_0603_1608Metric, F.Cu at (135.9, 108.4)
- added R61: 1k, Resistor_SMD:R_0603_1608Metric, F.Cu at (135.9, 110.9)
- added R62: 10k, Resistor_SMD:R_0603_1608Metric, F.Cu at (135.9, 113.4)
- added R63: 0.51k, Resistor_SMD:R_0603_1608Metric, F.Cu at (135.9, 115.9)
- added R64: 3.3k, Resistor_SMD:R_0603_1608Metric, F.Cu at (135.9, 118.5)
- added R65: 0.001, Resistor_SMD:R_2512_6332Metric, F.Cu at (133.7, 128.7)
- added R66: 0.001, Resistor_SMD:R_2512_6332Metric, F.Cu at (133.7, 133.6)
- added R7: 10k, Resistor_SMD:R_0603_1608Metric, F.Cu at (111.4, 90.9)
- added R8: 10K, Resistor_SMD:R_0603_1608Metric, F.Cu at (111.4, 93.4)
- added R9: 10K, Resistor_SMD:R_0603_1608Metric, F.Cu at (111.4, 95.9)
- added RN2: 10k, Resistor_SMD:R_Array_Concave_4x0603, F.Cu at (120.1, 97.1)
- added SW2: SW_Push, Button_Switch_SMD:SW_SPST_PTS810, F.Cu at (137.1, 87.0)
- added SW3: SW_Push, Button_Switch_SMD:SW_SPST_PTS810, F.Cu at (137.1, 91.8)
- added U1: HX711, Package_SO:SOP-16_3.9x9.9mm_P1.27mm, F.Cu at (193.8, 100.3)
- added U11: INA240A2PW, Package_SO:TSSOP-8_4.4x3mm_P0.65mm, F.Cu at (101.7, 144.9)
- added U3: ESP32-S3-WROOM-1, RF_Module:ESP32-S3-WROOM-1, F.Cu at (114.1, 70.7)
- added U4: LMR16030SDDAR, Package_SO:TI_SO-PowerPAD-8_ThermalVias, F.Cu at (69.0, 53.7)
- added U5: LMR16030SDDAR, Package_SO:TI_SO-PowerPAD-8_ThermalVias, F.Cu at (69.0, 60.4)
- added current1: current info, Connector_PinHeader_2.54mm:PinHeader_1x04_P2.54mm_Vertical, F.Cu at (180.0, 68.8)
- added current2: current info, Connector_PinHeader_2.54mm:PinHeader_1x04_P2.54mm_Vertical, F.Cu at (127.0, 128.6)
- added hall1: sig, Connector_PinHeader_2.54mm:PinHeader_1x03_P2.54mm_Vertical, F.Cu at (180.0, 81.1)
- added hall2: sig, Connector_PinHeader_2.54mm:PinHeader_1x03_P2.54mm_Vertical, F.Cu at (127.0, 140.8)
- added motor1: input, Connector_PinHeader_2.54mm:PinHeader_1x03_P2.54mm_Vertical, F.Cu at (184.6, 81.1)
- added motor2: input, Connector_PinHeader_2.54mm:PinHeader_1x03_P2.54mm_Vertical, F.Cu at (131.7, 140.8)
- C25: value 4.7uf/50v -> 100nf/50v; footprint Capacitor_SMD:C_1206_3216Metric -> Capacitor_SMD:C_0603_1608Metric
- C26: value 4.7uf/50v -> 1nF; footprint Capacitor_SMD:C_1206_3216Metric -> Capacitor_SMD:C_0603_1608Metric
- C27: value 100nf/50v -> 100nF
- C28: value 10uf/50v -> 330uf; footprint Capacitor_SMD:C_1210_3225Metric -> Capacitor_SMD:CP_Elec_10x10.5
- C29: value 100nf/50v -> 330uf; footprint Capacitor_SMD:C_0603_1608Metric -> Capacitor_SMD:CP_Elec_10x10.5
- C30: value 10uf/50v -> 100nF; footprint Capacitor_SMD:C_1210_3225Metric -> Capacitor_SMD:C_0603_1608Metric
- C31: value 68nF -> 20pF
- C32: value 47nF -> 1nF
- C33: value 47nF -> 100nF
- C34: value 100nF/16v -> 100nF
- C35: value 100nF/16v -> 20pF
- C36: value 100nF/16v -> 1nF
- C37, C38: value 10uF/35v -> 100nF; footprint Capacitor_SMD:C_1210_3225Metric -> Capacitor_SMD:C_0603_1608Metric
- C39: value 10uF/16v -> 20pF; footprint Capacitor_SMD:C_1210_3225Metric -> Capacitor_SMD:C_0603_1608Metric
- C40: value 10uF/16v -> 0.1nF; footprint Capacitor_SMD:C_1210_3225Metric -> Capacitor_SMD:C_0603_1608Metric
- C41: value 10uF/10v -> 0.1nF
- C42: value 10uF/10v -> 1uF
- C43: value 10uF -> 1uF
- C44: value 0.1uF -> 1nF
- C47: value 1uF(105) -> 330uf; footprint Capacitor_SMD:C_0402_1005Metric -> Capacitor_SMD:CP_Elec_10x10.5
- C48: value 10uF -> 330uf; footprint Capacitor_SMD:C_1206_3216Metric -> Capacitor_SMD:CP_Elec_10x10.5
- C49: value 1uF(105) -> 100nF; footprint Capacitor_SMD:C_0402_1005Metric -> Capacitor_SMD:C_0603_1608Metric
- C50: value 1uF(105) -> 20pF; footprint Capacitor_SMD:C_0402_1005Metric -> Capacitor_SMD:C_0603_1608Metric
- C51: value 1uF(105) -> 1nF; footprint Capacitor_SMD:C_0402_1005Metric -> Capacitor_SMD:C_0603_1608Metric
- C52, C53: value 10uF -> 100nF; footprint Capacitor_SMD:C_1206_3216Metric -> Capacitor_SMD:C_0603_1608Metric
- J2: value sig_in -> pa1010d; footprint Connector_PinHeader_2.54mm:PinHeader_1x02_P2.54mm_Vertical -> Connector_PinSocket_2.54mm:PinSocket_1x05_P2.54mm_Vertical
- J3: value sig_out -> can_sensor; footprint Connector_PinHeader_2.54mm:PinHeader_1x02_P2.54mm_Vertical -> TerminalBlock:TerminalBlock_MaiXu_MX126-5.0-04P_1x04_P5.00mm
- J4: value Conn_02x02_Counter_Clockwise -> USB_C_Receptacle_USB2.0_16P; footprint Connector_PinHeader_2.54mm:PinHeader_2x02_P2.54mm_Vertical -> Connector_USB:USB_C_Receptacle_G-Switch_GT-USB-7010ASV
- L1: value 22uH -> 47uH
- L2: value 47uH -> 22uH
- U10: value SIT1042AQT/3 -> INA240A2PW; footprint Package_DFN_QFN:DFN-8-1EP_3x3mm_P0.65mm_EP1.5x2.25mm -> Package_SO:TSSOP-8_4.4x3mm_P0.65mm
- U2: value TSSOP28-SH3676010B -> SIT1042AQT/3; footprint lceda:IC-TSSOP-28 -> Package_DFN_QFN:DFN-8-1EP_3x3mm_P0.65mm_EP1.5x2.25mm
- U7, U8: value LMR16030SDDAR -> INA240A2PW; footprint Package_SO:TI_SO-PowerPAD-8_ThermalVias -> Package_SO:TSSOP-8_4.4x3mm_P0.65mm
- moved J2 112.8 mm to (248.0, 57.4)
- moved C24 109.3 mm to (44.3, 60.9)
- moved C25 102.6 mm to (64.1, 33.3)
- moved L1 99.2 mm to (33.9, 34.4)
- moved L2 99.2 mm to (33.9, 48.7)
- moved L3 99.2 mm to (33.9, 63.0)
- moved SW1 92.3 mm to (202.9, 108.2)
- moved U6 85.0 mm to (69.0, 67.0)
- moved C40 84.2 mm to (180.8, 53.7)
- moved C39 82.7 mm to (180.8, 51.2)
- moved C38 81.2 mm to (180.8, 48.7)
- moved C37 79.7 mm to (180.8, 46.1)
- moved C36 79.6 mm to (180.8, 43.6)
- moved J3 75.0 mm to (212.4, 60.1)
- moved C30 71.9 mm to (176.8, 48.7)
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Connections:
- C24 pad 1: 24V/3A -> GND
- C24 pad 2: GND -> 24V/3A
- C25 pad 1: GND -> 24V/3A
- C25 pad 2: 24V/3A -> GND
- C26 pad 1: GND -> /foc1/A2
- C26 pad 2: 24V/3A -> GND
- C27 pad 1: 24V/3A -> Net-(Q4-SR)
- C28 pad 1: VIN_MAX60V -> VCC
- C29 pad 1: VIN_MAX60V -> VCC
- C30 pad 1: GND -> MOT_C
- C30 pad 2: VIN_MAX60V -> GND
- C31 pad 1: Net-(U6-SS/PGOOD) -> GND
- C31 pad 2: GND -> MOT_C
- C32 pad 1: Net-(U7-SS/PGOOD) -> /foc1/A3
- C33 pad 1: Net-(U8-SS/PGOOD) -> Net-(Q5-SR)
- C34 pad 1: 24V/3A -> MOT_A
- C34 pad 2: Net-(U6-BOOT) -> GND
- C35 pad 1: 5V/3A -> GND
- C35 pad 2: Net-(U7-BOOT) -> MOT_A
- C36 pad 1: 3.3V/3A -> Net-(Q6-IS)
- C36 pad 2: Net-(U8-BOOT) -> GND
- C37 pad 1: 24V/3A -> MOT_B
- C38 pad 1: GND -> Net-(Q6-SR)
- C38 pad 2: 24V/3A -> GND
- C39 pad 1: 5V/3A -> GND
- C39 pad 2: GND -> MOT_B
- C40 pad 1: GND -> Net-(U7-REF1)
- C40 pad 2: 5V/3A -> +3.3V
- C41 pad 1: 3.3V/3A -> Net-(U8-REF1)
- C41 pad 2: GND -> +3.3V
- C42 pad 1: GND -> EN
- C42 pad 2: 3.3V/3A -> GND
- C43 pad 1: GND -> IO0
- C43 pad 2: +3.3V -> GND
- C44 pad 1: Net-(U9-INA+) -> /foc2/A2
- C44 pad 2: Net-(U9-INA-) -> GND
- C47 pad 1: GND -> VCC
- C47 pad 2: EN -> GND
- C48 pad 1: +3.3V -> VCC
- C49 pad 1: GND -> MOT_C
- C49 pad 2: Net-(U13-VBUS) -> GND
- C50 pad 1: IO0 -> GND
- C50 pad 2: GND -> MOT_C
- C51 pad 1: EN -> /foc2/A3
- C52 pad 1: +5V -> Net-(Q8-SR)
- C53 pad 1: +5V -> MOT_A
- J2 pad 1: INA- -> +5V
- J2 pad 2: INA+ -> SDA
- J3 pad 1: DOUT -> GND
- J3 pad 2: PD_SCK -> 24V/3A
- L1 pad 1: Net-(D20-K) -> Net-(D11-K)
- L1 pad 2: 24V/3A -> +5V
- L2 pad 1: Net-(D21-K) -> Net-(D12-K)
- L2 pad 2: 5V/3A -> 24V/3A
- L3 pad 1: Net-(D22-K) -> Net-(D16-K)
- L3 pad 2: 3.3V/3A -> +3.3V
- U10 pad 1: TXD -> GND
- U10 pad 2: GND -> out1
- U10 pad 3: +5V -> out1_cs
- U10 pad 4: RXD -> GND
- U10 pad 6: CANL -> +3.3V
- U10 pad 7: CANH -> Net-(U10-REF1)
- U10 pad 8: GND -> /foc2/A0
- U2 pad 1: unconnected-(U2-NC0-Pad1) -> TXD_SENSOR
- U2 pad 2: <NO NET> -> GND
- U2 pad 3: <NO NET> -> +5V
- U2 pad 4: <NO NET> -> RXD_SENSOR
- U2 pad 5: <NO NET> -> +3.3V
- U2 pad 6: <NO NET> -> CANL
- U2 pad 7: <NO NET> -> CANH
- U2 pad 8: <NO NET> -> GND
- U2 pad 9: <NO NET> -> unconnected-(U2-EP-Pad9)
- U6 pad 2: VIN_MAX60V -> +5V
- U6 pad 8: Net-(D20-K) -> Net-(D16-K)
- U7 pad 1: Net-(U7-BOOT) -> GND
- U7 pad 2: 24V/3A -> out1
- U7 pad 3: unconnected-(U7-EN-Pad3) -> out1_cs
- U7 pad 4: Net-(U7-RT/YNC) -> GND
- U7 pad 5: Net-(U7-FB) -> +3.3V
- U7 pad 6: Net-(U7-SS/PGOOD) -> +3.3V
- U7 pad 7: GND -> Net-(U7-REF1)
- U7 pad 8: Net-(D21-K) -> /foc1/A0
- U8 pad 1: Net-(U8-BOOT) -> GND
- U8 pad 2: 24V/3A -> out3_cs
- U8 pad 3: unconnected-(U8-EN-Pad3) -> out3
- U8 pad 4: Net-(U8-RT/YNC) -> GND
- U8 pad 5: Net-(U8-FB) -> +3.3V
- U8 pad 6: Net-(U8-SS/PGOOD) -> +3.3V
- U8 pad 7: GND -> Net-(U8-REF1)
- U8 pad 8: Net-(D22-K) -> /foc1/A1
- U9 pad 11: PD_SCK -> PD_SCK2
- U9 pad 12: DOUT -> DOUT_2

Commit message: feat: update
Parts:
- removed the 3.3V2 at (34.4, 74.0)
- removed the 3.3V2 at (171.0, 84.5)
- removed the 3.3V4 at (118.1, 144.3)
- removed the 3.3V4 at (28.3, 74.0)
- removed the 42V2 at (171.0, 87.1)
- removed the 42V2 at (34.4, 76.6)
- removed 42V4: LED, LED_SMD:LED_0603_1608Metric
- removed the J1 at (243.4, 57.4)
- removed the J1 at (191.8, 108.4)
- removed the J8 at (196.5, 108.4)
- removed the J8 at (52.3, 67.7)
- removed current1, current2: current info, Connector_PinHeader_2.54mm:PinHeader_1x04_P2.54mm_Vertical
- removed hall1, hall2: sig, Connector_PinHeader_2.54mm:PinHeader_1x03_P2.54mm_Vertical
- removed motor1, motor2: input, Connector_PinHeader_2.54mm:PinHeader_1x03_P2.54mm_Vertical
- added 3.3V2: LED, LED_SMD:LED_0603_1608Metric, F.Cu at (146.8, 23.7)
- added 3.3V4: LED, LED_SMD:LED_0603_1608Metric, F.Cu at (156.1, 114.7)
- added 42V2: LED, LED_SMD:LED_0603_1608Metric, F.Cu at (146.8, 26.3)
- added J1: RC555, Connector_PinHeader_2.54mm:PinHeader_1x08_P2.54mm_Vertical, F.Cu at (374.9, 22.9)
- added J8: power, Connector_AMASS:AMASS_XT60PW-M_1x02_P7.20mm_Horizontal, F.Cu at (116.8, 100.2)
- moved Q1 261.3 mm to (363.3, 65.3)
- moved Q2 261.3 mm to (363.3, 69.9)
- moved Q3 261.3 mm to (363.3, 74.5)
- moved RN2 257.2 mm to (374.7, 60.2)
- moved J5 253.4 mm to (368.1, 65.2)
- moved D4 246.6 mm to (340.7, 66.7)
- moved D5 246.6 mm to (340.7, 74.5)
- moved D1 242.8 mm to (375.9, 63.8)
- moved D2 242.8 mm to (375.9, 65.8)
- moved D3 242.8 mm to (375.9, 67.7)
- moved C3 241.8 mm to (348.1, 64.1)
- moved C42 241.8 mm to (348.1, 66.6)
- moved C43 241.8 mm to (348.1, 69.1)
- moved C45 241.8 mm to (348.1, 71.7)
- moved R4 241.8 mm to (348.1, 74.2)
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Connections:
- U3 pad 17: MOT_C -> /mcu/MOT1_A
- U3 pad 18: MOT_B -> /mcu/MOT1_B
- U3 pad 19: MOT_A -> /mcu/MOT1_C
- U3 pad 20: MOT_A -> /mcu/MOT2_A
- U3 pad 21: MOT_B -> /mcu/MOT2_B
- U3 pad 22: MOT_C -> /mcu/MOT2_C

Commit message: feat: update
Parts:
- removed 3.3V2, 42V2, D19: LED, LED_SMD:LED_0603_1608Metric
- removed C21, C24: 4.7uf/50v, Capacitor_SMD:C_1206_3216Metric
- removed C28, C29: 330uf, Capacitor_SMD:CP_Elec_10x10.5
- removed Q2, Q3: SS8050, Package_TO_SOT_SMD:SOT-23
- removed R58: 1k, Resistor_SMD:R_0603_1608Metric
- removed R59, R64: 3.3k, Resistor_SMD:R_0603_1608Metric
- removed R8, R9: 10K, Resistor_SMD:R_0603_1608Metric
- C1, C10, C11, C12, C13, C18, C19, C2, C20, C22, C23, C25, C26, C27, C3, C30, C31, C32, C33, C36, C38, C4, C42, C44, C46, C49, C5, C50, C51, C52, C55, C57, C7, C8, C9, D1, D2, D3, Q1, R1, R10, R11, R12, R13, R14, R15, R16, R17, R18, R2, R21, R22, R24, R25, R26, R27, R28, R29, R30, R31, R32, R33, R34, R36, R38, R39, R4, R40, R41, R42, R43, R46, R47, R48, R49, R5, R50, R51, R52, R53, R54, R55, R57, R6, R60, R61, R62, R63, R7: moved to B.Cu
- C34, C37, C53, C56: value 100nF -> 20pF; moved to B.Cu
- C35, C39, C54, C58: value 20pF -> 100nF; moved to B.Cu
- C47, C48: value 330uf -> 220uf
- J1: footprint Connector_PinHeader_2.54mm:PinHeader_1x08_P2.54mm_Vertical -> Connector_JST:JST_PH_B8B-PH-K_1x08_P2.00mm_Vertical
- J11, J12, J3: footprint TerminalBlock:TerminalBlock_MaiXu_MX126-5.0-04P_1x04_P5.00mm -> Connector_JST:JST_PH_B4B-PH-K_1x04_P2.00mm_Vertical
- R35: value 10k -> 3.3k; moved to B.Cu
- R37: value 1k -> 3.3k; moved to B.Cu
- moved SW2 294.0 mm to (68.7, 119.8), turned to 180 degrees
- moved SW3 292.4 mm to (68.7, 115.0), turned to 180 degrees
- moved D1 283.8 mm to (96.9, 115.9), turned to 180 degrees
- moved J5 282.4 mm to (90.7, 117.9), turned to 180 degrees
- moved D2 282.3 mm to (96.8, 108.5), turned to -90 degrees
- moved C43 281.2 mm to (70.0, 110.6), turned to 180 degrees
- moved C45 280.5 mm to (70.0, 108.1), turned to 180 degrees
- moved D3 280.1 mm to (98.8, 108.5), turned to -90 degrees
- moved U1 262.6 mm to (88.3, 69.6), turned to 90 degrees
- moved D10 259.7 mm to (115.0, 106.3)
- moved D9 259.7 mm to (115.0, 103.7)
- moved D7 259.6 mm to (115.1, 100.9)
- moved D6 259.4 mm to (115.2, 97.6)
- moved RN2 256.9 mm to (120.8, 99.4)
- moved R5 255.6 mm to (99.8, 105.0), turned to -90 degrees
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Connections:
- C11 pad 1: Net-(U5-SS/PGOOD) -> Net-(U6-SS/PGOOD)
- C13 pad 2: Net-(U5-BOOT) -> Net-(U6-BOOT)
- C18 pad 1: Net-(U6-SS/PGOOD) -> Net-(U5-SS/PGOOD)
- C19 pad 2: Net-(U6-BOOT) -> Net-(U5-BOOT)
- C20 pad 1: 24V/3A -> GND
- C20 pad 2: GND -> 24V/3A
- C30 pad 1: MOT_C -> /foc1/MOT_A
- C31 pad 2: MOT_C -> /foc1/MOT_A
- C34 pad 1: MOT_A -> GND
- C34 pad 2: GND -> /foc1/MOT_B
- C35 pad 1: GND -> /foc1/MOT_B
- C35 pad 2: MOT_A -> GND
- C37 pad 1: MOT_B -> GND
- C37 pad 2: GND -> /foc2/MOT_B
- C39 pad 1: GND -> /foc2/MOT_B
- C39 pad 2: MOT_B -> GND
- C49 pad 1: MOT_C -> /foc2/MOT_A
- C50 pad 2: MOT_C -> /foc2/MOT_A
- C53 pad 1: MOT_A -> GND
- C53 pad 2: GND -> /foc1/MOT_C
- C54 pad 1: GND -> /foc1/MOT_C
- C54 pad 2: MOT_A -> GND
- C56 pad 1: MOT_B -> GND
- C56 pad 2: GND -> /foc2/MOT_C
- C58 pad 1: GND -> /foc2/MOT_C
- C58 pad 2: MOT_B -> GND
- J10 pad 2: MOT_A -> /foc2/MOT_A
- J10 pad 3: MOT_B -> /foc2/MOT_B
- J10 pad 4: MOT_C -> /foc2/MOT_C
- J7 pad 2: MOT_A -> /foc1/MOT_A
- J7 pad 3: MOT_B -> /foc1/MOT_B
- J7 pad 4: MOT_C -> /foc1/MOT_C
- L2 pad 1: Net-(D12-K) -> Net-(D16-K)
- L2 pad 2: 24V/3A -> +3.3V
- L3 pad 1: Net-(D16-K) -> Net-(D12-K)
- L3 pad 2: +3.3V -> 24V/3A
- R12 pad 1: Net-(U5-RT/YNC) -> Net-(U6-RT/YNC)
- R17 pad 2: Net-(U5-FB) -> Net-(U6-FB)
- R18 pad 1: Net-(U5-FB) -> Net-(U6-FB)
- R22 pad 1: Net-(U6-RT/YNC) -> Net-(U5-RT/YNC)
- R25 pad 2: Net-(U6-FB) -> Net-(U5-FB)
- R26 pad 1: Net-(U6-FB) -> Net-(U5-FB)
- R33 pad 1: MOT_C -> /foc1/MOT_A
- R35 pad 1: VCC -> /foc1/MOT_B
- R35 pad 2: Net-(42V2-A) -> +3.3V
- R37 pad 1: Net-(3.3V2-A) -> /foc2/MOT_B
- R38 pad 1: +3.3V -> /foc1/MOT_C
- R38 pad 2: MOT_A -> +3.3V
- R43 pad 1: MOT_B -> /foc2/MOT_C
- R54 pad 1: MOT_C -> /foc2/MOT_A
- U3 pad 17: /mcu/MOT1_A -> /foc1/MOT_C
- U3 pad 18: /mcu/MOT1_B -> /foc1/MOT_B
- U3 pad 19: /mcu/MOT1_C -> /foc1/MOT_A
- U3 pad 20: /mcu/MOT2_A -> /foc2/MOT_A
- U3 pad 21: /mcu/MOT2_B -> /foc2/MOT_B
- U3 pad 22: /mcu/MOT2_C -> /foc2/MOT_C
- U3 pad 28: PD_SCK2 -> /foc1/IN_3
- U3 pad 29: DOUT_1 -> /foc1/IN_2
- U3 pad 30: PD_SCK1 -> /foc1/IN_1
- U3 pad 31: /foc1/IN_1 -> PD_SCK2
- U3 pad 32: /foc1/IN_2 -> DOUT_1
- U3 pad 33: /foc1/IN_3 -> PD_SCK1
- U5 pad 2: VCC -> +5V
- U5 pad 8: Net-(D12-K) -> Net-(D16-K)
- U6 pad 2: +5V -> VCC
- U6 pad 8: Net-(D16-K) -> Net-(D12-K)

Commit message: feat: update
Parts:
- removed C47: 220uf, Capacitor_SMD:CP_Elec_10x10.5
- removed RN2: 10k, Resistor_SMD:R_Array_Concave_4x0603
- added J13: Conn_01x01_Pin, MountingHole:MountingHole_4.3mm_M4, F.Cu at (105.9, 83.5)
- added J14: Conn_01x01_Pin, MountingHole:MountingHole_4.3mm_M4, F.Cu at (134.2, 82.4)
- added J15: Conn_01x01_Pin, MountingHole:MountingHole_4.3mm_M4, F.Cu at (113.7, 142.3)
- added J16: Conn_01x01_Pin, MountingHole:MountingHole_4.3mm_M4, F.Cu at (166.8, 132.6)
- added R58: 10K, Resistor_SMD:R_0603_1608Metric, B.Cu at (146.8, 99.5)
- added R59: 10K, Resistor_SMD:R_0603_1608Metric, B.Cu at (143.9, 99.5)
- added R8: 10K, Resistor_SMD:R_0603_1608Metric, B.Cu at (152.7, 101.1)
- added R9: 10K, Resistor_SMD:R_0603_1608Metric, B.Cu at (149.6, 101.2)
- 3.3V4: value LED -> VCC
- C14, C15, C16, C17, C43, C45, D15, D4, D5, D8, R19, R20, R23: moved to B.Cu
- C40, C41: value 0.1nF -> 0.1uF; moved to B.Cu
- C59, C60: value 0.1nF -> 0.1uF
- D10: value LED -> TXD
- D13: value LED -> +24V
- D14: value LED -> +5V
- D17: value LED -> +3.3V
- D7: value 3.3v -> +3.3v
- D9: value LED -> RXD
- SW2: value SW_Push -> BOOT
- SW3: value SW_Push -> EN
- moved J8 159.8 mm to (102.5, 137.0)
- moved R56 152.5 mm to (109.9, 152.3)
- moved 3.3V4 147.7 mm to (109.9, 149.9)
- moved D11 136.8 mm to (114.8, 131.3), turned to -90 degrees
- moved U4 136.5 mm to (114.8, 122.3), turned to 0 degrees
- moved C20 131.1 mm to (113.8, 117.9), turned to 180 degrees
- moved R23 130.0 mm to (91.3, 117.3)
- moved L3 129.0 mm to (141.8, 146.4)
- moved D12 129.0 mm to (152.7, 148.5)
- moved C10 128.7 mm to (148.0, 131.2), turned to 0 degrees
- moved U6 127.8 mm to (153.6, 138.7)
- moved R15 127.4 mm to (118.5, 115.3), turned to 180 degrees
- moved D17 126.1 mm to (91.3, 117.3)
- moved R18 125.1 mm to (146.6, 137.9), turned to 90 degrees
- moved C25 125.0 mm to (110.2, 123.4)
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Connections:
- C12 pad 1: +5V -> /mcu/Battery_5V
- C14 pad 1: +5V -> /mcu/Battery_5V
- C15 pad 2: +5V -> /mcu/Battery_5V
- C40 pad 1: Net-(U7-REF1) -> GND
- C41 pad 1: Net-(U8-REF1) -> GND
- C59 pad 1: Net-(U10-REF1) -> GND
- C60 pad 1: Net-(U11-REF1) -> GND
- D13 pad 2: +24V -> 24V/3A
- D5 pad 2: +5V -> /mcu/Battery_5V
- J6 pad 1: out1 -> Net-(J6-Pin_1)
- J6 pad 2: out2 -> Net-(J6-Pin_2)
- J6 pad 3: out3 -> Net-(J6-Pin_3)
- J9 pad 1: out1 -> Net-(J9-Pin_1)
- J9 pad 2: out2 -> Net-(J9-Pin_2)
- J9 pad 3: out3 -> Net-(J9-Pin_3)
- L1 pad 2: +5V -> /mcu/Battery_5V
- Q1 pad 3: +5V -> /mcu/Battery_5V
- Q4 pad 4: out1_cs -> Net-(U7--)
- Q4 pad 8: out1_cs -> Net-(U7--)
- Q5 pad 4: out2 -> Net-(J6-Pin_2)
- Q5 pad 8: out2 -> Net-(J6-Pin_2)
- Q6 pad 4: out3_cs -> Net-(U8-+)
- Q6 pad 8: out3_cs -> Net-(U8-+)
- Q7 pad 4: out1_cs -> Net-(U10--)
- Q7 pad 8: out1_cs -> Net-(U10--)
- Q8 pad 4: out2 -> Net-(J9-Pin_2)
- Q8 pad 8: out2 -> Net-(J9-Pin_2)
- Q9 pad 4: out3_cs -> Net-(U11-+)
- Q9 pad 8: out3_cs -> Net-(U11-+)
- R13 pad 1: +5V -> /mcu/Battery_5V
- R44 pad 1: out1 -> Net-(J6-Pin_1)
- R44 pad 2: out1_cs -> Net-(U7--)
- R45 pad 1: out3_cs -> Net-(U8-+)
- R45 pad 2: out3 -> Net-(J6-Pin_3)
- R65 pad 1: out1 -> Net-(J9-Pin_1)
- R65 pad 2: out1_cs -> Net-(U10--)
- R66 pad 1: out3_cs -> Net-(U11-+)
- R66 pad 2: out3 -> Net-(J9-Pin_3)
- U10 pad 2: out1 -> Net-(J9-Pin_1)
- U10 pad 3: out1_cs -> Net-(U10--)
- U10 pad 7: Net-(U10-REF1) -> GND
- U11 pad 2: out3_cs -> Net-(U11-+)
- U11 pad 3: out3 -> Net-(J9-Pin_3)
- U11 pad 7: Net-(U11-REF1) -> GND
- U3 pad 17: /foc1/MOT_C -> /foc1/IN_3
- U3 pad 18: /foc1/MOT_B -> /foc1/IN_2
- U3 pad 19: /foc1/MOT_A -> /foc1/IN_1
- U3 pad 20: /foc2/MOT_A -> /foc2/IN_3
- U3 pad 21: /foc2/MOT_B -> /foc2/IN_2
- U3 pad 22: /foc2/MOT_C -> /foc2/IN_1
- U3 pad 26: /foc2/IN_3 -> /foc1/MOT_C
- U3 pad 28: /foc1/IN_3 -> /foc2/MOT_C
- U3 pad 29: /foc1/IN_2 -> /foc2/MOT_B
- U3 pad 30: /foc1/IN_1 -> /foc2/MOT_A
- U3 pad 34: /foc2/IN_1 -> /foc1/MOT_A
- U3 pad 35: /foc2/IN_2 -> /foc1/MOT_B
- U7 pad 2: out1 -> Net-(J6-Pin_1)
- U7 pad 3: out1_cs -> Net-(U7--)
- U7 pad 7: Net-(U7-REF1) -> GND
- U8 pad 2: out3_cs -> Net-(U8-+)
- U8 pad 3: out3 -> Net-(J6-Pin_3)
- U8 pad 7: Net-(U8-REF1) -> GND
Routing:
- net +3.3V: track 0.00 -> 404.8 mm, vias 0 -> 14
- net +5V: track 0.00 -> 182.3 mm, vias 0 -> 4
- net 24V/3A: track 0.00 -> 123.2 mm, vias 0 -> 3
- net /mcu/Battery_5V: track 0.00 -> 79.6 mm, vias 0 -> 3
- net SDA: track 0.00 -> 67.5 mm
- net VBUS: track 0.00 -> 67.2 mm, vias 0 -> 1
- net SCK: track 0.00 -> 58.3 mm
- net /foc2/IN_3: track 0.00 -> 45.6 mm, vias 0 -> 2
- net U0_TXD: track 0.00 -> 43.0 mm, vias 0 -> 1
- net /foc1/IN_1: track 0.00 -> 40.7 mm, vias 0 -> 2
- net GND: track 0.00 -> 39.7 mm, vias 0 -> 88
- net /foc2/IN_2: track 0.00 -> 33.9 mm, vias 0 -> 2
- net U0_RXD: track 0.00 -> 33.5 mm, vias 0 -> 1
- net /foc1/IN_2: track 0.00 -> 30.5 mm, vias 0 -> 2
- net Net-(D12-K): track 0.00 -> 29.5 mm
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- added copper zone on B.Cu, net GND
- added copper zone on F.Cu, net Net-(J6-Pin_1)
- added copper zone on F.Cu, net Net-(J6-Pin_2)
- added copper zone on F.Cu, net Net-(J6-Pin_3)
- added copper zone on F.Cu, net Net-(J9-Pin_1)
- added copper zone on F.Cu, net Net-(J9-Pin_2)
- added copper zone on F.Cu, net Net-(J9-Pin_3)
- added copper zone on F.Cu, net Net-(U10--)
- added copper zone on F.Cu, net Net-(U11-+)
- added copper zone on F.Cu, net Net-(U7--)
- added copper zone on F.Cu, net Net-(U8-+)
- added copper zone on F.Cu, net VCC
Other:
- board outline added: 86.2 x 84.8 mm
- copper layers 2 -> 4

Commit message: feat: update
Parts:
- C40, C41, C59, C60: value 0.1uF -> 100nF
- moved D15 6.12 mm to (114.8, 85.7)
- moved D8 6.12 mm to (114.8, 89.5)
- moved R2 3.42 mm to (135.8, 93.7)
- moved C1 2.76 mm to (133.1, 89.7), turned to -90 degrees
- moved R4 1.55 mm to (159.7, 143.5)
- moved R3 1.19 mm to (112.7, 79.5), turned to 180 degrees
- moved R1 0.70 mm to (135.8, 95.3)
- turned C2 to 0 degrees
Connections:
- R27 pad 2: +3.3V -> MOTO_POWER
- R31 pad 2: +3.3V -> MOTO_POWER
- R39 pad 2: +3.3V -> MOTO_POWER
- R48 pad 2: +3.3V -> MOTO_POWER
- R52 pad 2: +3.3V -> MOTO_POWER
- R60 pad 2: +3.3V -> MOTO_POWER
- U2 pad 9: unconnected-(U2-EP-Pad9) -> GND
- U3 pad 12: /foc2/A1 -> MOSI
- U3 pad 16: unconnected-(U3-IO46-Pad16) -> MOTO_POWER
- U3 pad 23: DOUT_2 -> PD_SCK2
- U3 pad 24: unconnected-(U3-IO47-Pad24) -> DOUT_2
- U3 pad 26: /foc1/MOT_C -> unconnected-(U3-IO45-Pad26)
- U3 pad 31: PD_SCK2 -> /foc1/MOT_A
- U3 pad 32: DOUT_1 -> SDA
- U3 pad 33: PD_SCK1 -> SCK
- U3 pad 34: /foc1/MOT_A -> /foc1/MOT_B
- U3 pad 35: /foc1/MOT_B -> /foc1/MOT_C
- U3 pad 38: IRQ -> RST
- U3 pad 39: RST -> IRQ
- U3 pad 4: MOSI -> /foc1/A1
- U3 pad 6: /foc1/A1 -> /foc2/A0
- U3 pad 7: /foc2/A0 -> /foc2/A1
- U3 pad 8: SCK -> PD_SCK1
- U3 pad 9: SDA -> DOUT_1
Routing:
- net IRQ: track 0.00 -> 93.1 mm, vias 0 -> 2
- net MOTO_POWER: track 0.00 -> 89.7 mm, vias 0 -> 3
- net RST: track 0.00 -> 89.0 mm, vias 0 -> 2
- net MOSI: track 0.00 -> 67.7 mm, vias 0 -> 1
- net SCK: track 58.3 -> 125.1 mm, vias 0 -> 1
- net /foc1/MOT_B: track 5.96 -> 72.4 mm, vias 1 -> 2
- net MISO: track 0.00 -> 66.3 mm, vias 0 -> 1
- net /foc1/MOT_C: track 6.92 -> 72.5 mm, vias 1 -> 2
- net /foc1/MOT_A: track 6.73 -> 72.1 mm, vias 1 -> 2
- net USB_D-: track 3.46 -> 67.8 mm, vias 1 -> 2
- net SDA: track 67.5 -> 130.7 mm, vias 0 -> 1
- net /foc1/A0: track 0.00 -> 62.7 mm, vias 0 -> 2
- net USB_D+: track 4.36 -> 66.9 mm, vias 1 -> 2
- net /foc1/A1: track 0.00 -> 62.3 mm, vias 0 -> 2
- net EN: track 26.3 -> 84.3 mm
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Other:
- outline, holes or cut-outs redrawn
