File: pcb/skateboard.kicad_pcb (KiCad board)
At the start: 4 copper layers, 86.2 x 84.8 mm, 177 parts, among them J1 RC555, J10 PH_2.0, J11 adc_sensor2, J12 adc_sensor1, J13 Conn_01x01_Pin, J14 Conn_01x01_Pin, J15 Conn_01x01_Pin, J16 Conn_01x01_Pin, J2 pa1010d, J3 can_sensor, J4 USB_C_Receptacle_USB2.0_16P, J5 UART, J6 TB_MOTOR, J7 PH_2.0, J8 power, J9 TB_MOTOR, Q1 AO3401A, Q4 BTN8982TA, Q5 BTN8982TA, Q6 BTN8982TA, Q7 BTN8982TA, Q8 BTN8982TA, Q9 BTN8982TA, SW1 SW_SPST, SW2 BOOT, SW3 EN, U1 HX711, U10 INA240A2PW, U11 INA240A2PW, U2 SIT1042AQT/3, U3 ESP32-S3-WROOM-1, U4 LMR16030SDDAR, U5 LMR16030SDDAR, U6 LMR16030SDDAR, U7 INA240A2PW, U8 INA240A2PW, U9 HX711

Commit message: update
Parts:
- added C21: 100nf, Capacitor_SMD:C_0603_1608Metric, B.Cu at (137.9, 84.7)
- added C24: 100nf, Capacitor_SMD:C_0603_1608Metric, B.Cu at (142.8, 82.2)
- added C28: 100nf, Capacitor_SMD:C_0603_1608Metric, B.Cu at (137.9, 86.2)
- added C6: 100nf, Capacitor_SMD:C_0603_1608Metric, B.Cu at (142.8, 83.8)
- added R64: 200k, Resistor_SMD:R_0603_1608Metric, F.Cu at (94.0, 91.3)
- added R67: 200k, Resistor_SMD:R_0603_1608Metric, F.Cu at (168.1, 129.3)
- added R68: 200k, Resistor_SMD:R_0603_1608Metric, F.Cu at (99.0, 115.1)
- added R69: 200k, Resistor_SMD:R_0603_1608Metric, B.Cu at (159.0, 108.1)
- C12, C13, C19: value 100nF/16v -> 100nF
- C40, C41: moved to F.Cu
- C59, C60: moved to B.Cu
- C8: value 100nf/50v -> 100nf
- D4, D5: value MBR120VLSFT1G -> B560C
- moved SW2 76.8 mm to (93.8, 112.7), turned to 0 degrees
- moved SW3 68.8 mm to (93.7, 117.9), turned to 0 degrees
- moved C43 46.1 mm to (109.8, 150.4), turned to 0 degrees
- moved D4 41.4 mm to (115.0, 102.1), turned to 180 degrees
- moved C15 41.2 mm to (105.0, 109.0)
- moved C14 41.2 mm to (104.9, 112.7)
- moved R7 41.2 mm to (112.6, 107.9), turned to 90 degrees
- moved D5 40.2 mm to (115.0, 95.1), turned to 180 degrees
- moved C45 31.6 mm to (133.3, 150.5), turned to 0 degrees
- moved Q1 31.0 mm to (116.1, 107.9), turned to 0 degrees
- moved R19 28.5 mm to (136.5, 148.0), turned to -90 degrees
- moved 3.3V4 23.3 mm to (90.4, 137.2), turned to -90 degrees
- moved R56 22.7 mm to (90.4, 140.8), turned to 90 degrees
- moved D14 11.0 mm to (109.8, 122.9), turned to -90 degrees
- moved D17 10.7 mm to (101.9, 119.2), turned to 90 degrees
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Connections:
- Q4 pad 4: Net-(U7--) -> Net-(U7-+)
- Q4 pad 8: Net-(U7--) -> Net-(U7-+)
- Q6 pad 4: Net-(U8-+) -> Net-(U8--)
- Q6 pad 8: Net-(U8-+) -> Net-(U8--)
- Q7 pad 4: Net-(U10--) -> Net-(U10-+)
- Q7 pad 8: Net-(U10--) -> Net-(U10-+)
- Q9 pad 4: Net-(U11-+) -> Net-(U11--)
- Q9 pad 8: Net-(U11-+) -> Net-(U11--)
- R44 pad 2: Net-(U7--) -> Net-(U7-+)
- R45 pad 1: Net-(U8-+) -> Net-(U8--)
- R65 pad 2: Net-(U10--) -> Net-(U10-+)
- R66 pad 1: Net-(U11-+) -> Net-(U11--)
- U10 pad 2: Net-(J9-Pin_1) -> Net-(U10-+)
- U10 pad 3: Net-(U10--) -> Net-(J9-Pin_1)
- U10 pad 6: +3.3V -> Net-(U10-REF2)
- U11 pad 2: Net-(U11-+) -> Net-(J9-Pin_3)
- U11 pad 3: Net-(J9-Pin_3) -> Net-(U11--)
- U11 pad 6: +3.3V -> Net-(U11-REF2)
- U7 pad 2: Net-(J6-Pin_1) -> Net-(U7-+)
- U7 pad 3: Net-(U7--) -> Net-(J6-Pin_1)
- U7 pad 6: +3.3V -> Net-(U7-REF2)
- U8 pad 2: Net-(U8-+) -> Net-(J6-Pin_3)
- U8 pad 3: Net-(J6-Pin_3) -> Net-(U8--)
- U8 pad 6: +3.3V -> Net-(U8-REF2)
Routing:
- net +3.3V: track 379.5 -> 273.0 mm, vias 14 -> 9
- net +5V: track 217.4 -> 159.7 mm, vias 4 -> 2
- net EN: track 84.3 -> 37.4 mm, vias 2 -> 1
- net GND: track 51.5 -> 12.3 mm, vias 90 -> 76
- net TXD_SENSOR: track 38.4 -> 0.00 mm
- net Net-(D16-K): track 25.5 -> 0.00 mm, vias 3 -> 0
- net Net-(U10--): track 23.4 -> 0.00 mm
- net Net-(U8-+): track 23.0 -> 0.00 mm
- net Net-(U7--): track 20.8 -> 0.00 mm
- net /foc2/A1: track 57.2 -> 38.5 mm
- net Net-(D12-K): track 29.5 -> 10.9 mm
- net /mcu/Battery_5V: track 80.2 -> 62.4 mm, vias 3 -> 2
- net Net-(U11-+): track 14.2 -> 0.00 mm
- net Net-(U8--): track 0.00 -> 13.6 mm
- net Net-(U10-+): track 0.00 -> 13.5 mm
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- removed copper zone on F.Cu, net Net-(J6-Pin_1)
- removed copper zone on F.Cu, net Net-(J6-Pin_2)
- removed copper zone on F.Cu, net Net-(J6-Pin_3)
- removed copper zone on F.Cu, net Net-(J9-Pin_1)
- removed copper zone on F.Cu, net Net-(J9-Pin_2)
- removed copper zone on F.Cu, net Net-(J9-Pin_3)
- removed copper zone on F.Cu, net Net-(U10--)
- removed copper zone on F.Cu, net Net-(U11-+)
- removed copper zone on F.Cu, net Net-(U7--)
- removed copper zone on F.Cu, net Net-(U8-+)
Other:
- board size 86.2 x 84.8 mm -> 83.6 x 84.8 mm

Commit message: update
Parts:
- added J17: Conn_01x02_Pin, Connector_PinSocket_2.54mm:PinSocket_1x02_P2.54mm_Vertical, F.Cu at (169.6, 133.0)
- C40, R68: moved to B.Cu
- C59: moved to F.Cu
- moved C40 66.0 mm to (98.3, 115.0), turned to 0 degrees
- moved C59 64.6 mm to (163.5, 108.3), turned to -90 degrees
- moved C45 51.1 mm to (94.9, 116.7), turned to 180 degrees
- moved C43 41.5 mm to (95.0, 111.7), turned to 180 degrees
- moved D13 17.1 mm to (137.3, 138.8)
- moved R23 17.1 mm to (107.4, 123.0), turned to -90 degrees
- moved R10 14.0 mm to (109.0, 124.9), turned to -90 degrees
- moved C42 13.7 mm to (142.8, 80.6), turned to 0 degrees
- moved C10 13.6 mm to (157.6, 142.9), turned to 90 degrees
- moved R6 12.8 mm to (142.8, 79.0)
- moved R13 11.8 mm to (122.4, 122.4)
- moved C14 11.4 mm to (115.4, 117.3)
- moved C15 11.4 mm to (115.4, 113.5)
- moved R11 11.2 mm to (111.4, 124.2), turned to 180 degrees
- moved C8 11.0 mm to (160.1, 140.7)
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Connections:
- U3 pad 23: PD_SCK2 -> DOUT_2
- U3 pad 24: DOUT_2 -> PD_SCK2
- U3 pad 25: unconnected-(U3-IO48-Pad25) -> Battery_RXD
- U3 pad 26: unconnected-(U3-IO45-Pad26) -> Battery_TXD
Routing:
- net VBUS: track 66.2 -> 143.0 mm, vias 2 -> 3
- net EN: track 37.4 -> 97.1 mm, vias 1 -> 2
- net +5V: track 159.7 -> 208.0 mm, vias 2 -> 5
- net Battery_RXD: track 0.00 -> 48.3 mm, vias 0 -> 1
- net Battery_TXD: track 0.00 -> 43.6 mm, vias 0 -> 1
- net GND: track 12.3 -> 51.6 mm, vias 76 -> 89
- net TXD_SENSOR: track 0.00 -> 32.5 mm
- net Net-(D16-K): track 0.00 -> 28.7 mm, vias 0 -> 3
- net +3.3V: track 273.0 -> 300.0 mm, vias 9 -> 13
- net RXD_SENSOR: track 45.5 -> 26.0 mm, vias 1 -> 2
- net /foc2/A1: track 38.5 -> 54.4 mm
- net Net-(U4-RT/YNC): track 14.9 -> 0.00 mm
- net INA2+: track 14.4 -> 2.08 mm
- net Net-(SW1-A): track 14.4 -> 2.29 mm
- net INA2-: track 12.0 -> 2.13 mm
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- added copper zone on In1.Cu, net GND
- added copper zone on F.Cu, net Net-(J6-Pin_1)
- added copper zone on F.Cu, net Net-(J6-Pin_2)
- added copper zone on F.Cu, net Net-(J6-Pin_3)
- added copper zone on F.Cu, net Net-(J9-Pin_1)
- added copper zone on F.Cu, net Net-(J9-Pin_2)
- added copper zone on F.Cu, net Net-(J9-Pin_3)
- added copper zone on F.Cu, net Net-(U10-+)
- added copper zone on F.Cu, net Net-(U11--)
- added copper zone on F.Cu, net Net-(U7-+)
- added copper zone on F.Cu, net Net-(U8--)
- added copper zone on In2.Cu, net VCC

Commit message: feat: update
Routing:
- net MOTO_POWER: track 85.8 -> 84.5 mm
Changed lines of the file:
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@@
 			(drillshape 0)
 			(scaleselection 1)
-			(outputdirectory "C:/Users/Aril Linda/Desktop/millionBoard/pcb/Gerber/")
+			(outputdirectory "C:/Users/Aril Linda/Desktop/millionBoard/pcb/Gerber")
 		)
 	)
@@
 		(tags "Through hole socket strip THT 1x02 2.54mm single row")
 		(property "Reference" "J17"
-			(at 0 -2.77 0)
+			(at -2.8448 -0.254 0)
 			(layer "F.SilkS")
 			(effects
@@
 		(tags "Through hole socket strip THT 1x05 2.54mm single row")
 		(property "Reference" "J2"
-			(at 0 -2.77 0)
+			(at -2.6812 -0.1088 0)
 			(layer "F.SilkS")
 			(effects
@@
 	)
 	(via
-		(at 140.505 83.52)
+		(at 140.5065 83.5215)
 		(size 0.6)
 		(drill 0.3)
@@
 	(segment
 		(start 140.775 83.79)
-		(end 140.505 83.52)
+		(end 140.5065 83.5215)
 		(width 0.2)
 		(layer "B.Cu")
@@
 	)
 	(segment
-		(start 122.3401 83.8654)
-		(end 121.7568 84.4487)
+		(start 140.5065 83.5215)
+		(end 140.505 83.52)
 		(width 0.2)
-		(layer "In2.Cu")
+		(layer "B.Cu")
 		(net 37)
 	)
 	(segment
-		(start 132.9133 85.322)
-		(end 131.4567 83.8654)
+		(start 138.555958 85.322)
+		(end 140.357957 83.52)
 		(width 0.2)
 		(layer "In2.Cu")
@@
 	)
 	(segment
-		(start 139.523379 84.354579)
-		(end 140.089957 83.788)
+		(start 122.3401 83.8654)
+		(end 121.7568 84.4487)
 		(width 0.2)
 		(layer "In2.Cu")
@@
 	)
 	(segment
-		(start 121.7568 91.449743)
-		(end 101.5492 111.657343)
+		(start 132.9133 85.322)
+		(end 131.4567 83.8654)
 		(width 0.2)
 		(layer "In2.Cu")
@@
 	)
 	(segment
-		(start 139.523379 84.354579)
-		(end 138.555958 85.322)
+		(start 121.7568 91.449743)
+		(end 101.5492 111.657343)
 		(width 0.2)
 		(layer "In2.Cu")
@@
 	)
 	(segment
-		(start 139.503 84.374957)
-		(end 139.523379 84.354579)
-		(width 0.2)
-		(layer "In2.Cu")
-		(net 37)
-	)
-	(segment
 		(start 101.5492 111.657343)
 		(end 101.5492 112.685729)
@@
 	)
 	(segment
-		(start 140.505 83.788)
+		(start 140.357957 83.52)
 		(end 140.505 83.52)
 		(width 0.2)
@@
 	)
 	(segment
-		(start 140.089957 83.788)
-		(end 140.505 83.788)
-		(width 0.2)
-		(layer "In2.Cu")
-		(net 37)
-	)
-	(segment
 		(start 161.5225 107.32)
 		(end 160.2436 107.32)
@@
 		(width 0.2)
 		(layer "B.Cu")
-		(net 134)
-	)
-	(segment
-		(start 140.104 125.19)
-		(end 140.104 126.51)
-		(width 0.2)
-		(layer "B.Cu")
