File: pcb/skateboard.kicad_pcb (KiCad board)
At the start: 4 copper layers, 83.6 x 84.8 mm, 186 parts, among them J1 RC555, J10 PH_2.0, J11 adc_sensor2, J12 adc_sensor1, J13 Conn_01x01_Pin, J14 Conn_01x01_Pin, J15 Conn_01x01_Pin, J16 Conn_01x01_Pin, J17 Conn_01x02_Pin, J2 pa1010d, J3 can_sensor, J4 USB_C_Receptacle_USB2.0_16P, J5 UART, J6 TB_MOTOR, J7 PH_2.0, J8 power, J9 TB_MOTOR, Q1 AO3401A, Q4 BTN8982TA, Q5 BTN8982TA, Q6 BTN8982TA, Q7 BTN8982TA, Q8 BTN8982TA, Q9 BTN8982TA, SW1 SW_SPST, SW2 BOOT, SW3 EN, U1 HX711, U10 INA240A2PW, U11 INA240A2PW, U2 SIT1042AQT/3, U3 ESP32-S3-WROOM-1, U4 LMR16030SDDAR, U5 LMR16030SDDAR, U6 LMR16030SDDAR, U7 INA240A2PW, U8 INA240A2PW, U9 HX711

Commit message: feat: new_dc-dc pcb
Parts:
- L2: value 22uH -> 10uH
Changed lines of the file:
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@@
 (kicad_pcb
-	(version 20250324)
+	(version 20250401)
 	(generator "pcbnew")
 	(generator_version "9.99")
@@
 			)
 		)
-		(property "Value" "22uH"
+		(property "Value" "10uH"
 			(at 0 7.25 90)
 			(layer "F.Fab")
@@
 		)
 		(initial_side "right")
+		(is_time_domain no)
 		(last_diff_pair_gap 0.25)
 		(last_netname "INA1-")
@@
 		(rounded yes)
 		(single_sided no)
+		(target_delay 1000000)
+		(target_delay_max 1000000)
+		(target_delay_min 0)
 		(target_length 1000000)
 		(target_length_max 1000000)
