File: pcb/skateboard.kicad_sch (KiCad schematic)
At the start: 0 parts

Commit message: feat: update
Other:
- removed sheet GPS和音频
- removed sheet ad转换
- removed sheet dc-dc
- removed sheet 电机驱动
- removed sheet 电池保护
- added sheet power (dc-dc/dc-dc.kicad_sch)
- added sheet sensor (sensor/sensor.kicad_sch)
Changed lines of the file:
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@@
 (kicad_sch
-	(version 20231120)
+	(version 20250227)
 	(generator "eeschema")
-	(generator_version "8.0")
+	(generator_version "9.99")
 	(paper "A2")
 	(sheet
-		(at 74.93 102.87)
-		(size 67.31 53.34)
+		(at 232.41 88.9)
+		(size 52.07 45.72)
+		(exclude_from_sim no)
+		(in_bom yes)
+		(on_board yes)
+		(dnp no)
 		(fields_autoplaced yes)
 		(stroke
@@
 			(color 0 0 0 0.0000)
 		)
-		(property "Sheetname" "电池保护"
-			(at 74.93 102.1584 0)
+		(property "Sheetname" "sensor"
+			(at 232.41 88.1884 0)
 			(effects
 				(font
@@
 			)
 		)
-		(property "Sheetfile" "battery_protect.kicad_sch"
-			(at 74.93 156.7946 0)
+		(property "Sheetfile" "sensor/sensor.kicad_sch"
+			(at 232.41 135.2046 0)
 			(effects
 				(font
@@
 			(project "skateboard"
 				(path "/5cdb5c16-5e05-458b-86f0-906cf8114d7e"
-					(page "3")
+					(page "4")
+				)
+			)
+		)
+	)
+	(sheet
+		(at 345.44 109.22)
+		(size 60.96 43.18)
+		(exclude_from_sim no)
+		(in_bom yes)
+		(on_board yes)
+		(dnp no)
+		(fields_autoplaced yes)
+		(stroke
+			(width 0.1524)
+			(type solid)
+		)
+		(fill
+			(color 0 0 0 0.0000)
+		)
+		(property "Sheetname" "power"
+			(at 345.44 108.5084 0)
+			(effects
+				(font
+					(size 1.27 1.27)
+				)
+				(justify left bottom)
+			)
+		)
+		(property "Sheetfile" "dc-dc/dc-dc.kicad_sch"
+			(at 345.44 152.9846 0)
+			(effects
+				(font
+					(size 1.27 1.27)
+				)
+				(justify left top)
+			)
+		)
+		(instances
+			(project "skateboard"
+				(path "/5cdb5c16-5e05-458b-86f0-906cf8114d7e"
+					(page "5")
 				)
 			)
@@
 		(at 194.056 212.852)
 		(size 69.85 61.214)
+		(exclude_from_sim no)
+		(in_bom yes)
+		(on_board yes)
+		(dnp no)
 		(fields_autoplaced yes)
 		(stroke
@@
 		)
 	)
-	(sheet
-		(at 305.054 107.442)
-		(size 78.486 51.308)
-		(fields_autoplaced yes)
-		(stroke
-			(width 0.1524)
-			(type solid)
-		)
-		(fill
-			(color 0 0 0 0.0000)
-		)
-		(property "Sheetname" "电机驱动"
-			(at 305.054 106.7304 0)
-			(effects
-				(font
-					(size 1.27 1.27)
-				)
-				(justify left bottom)
-			)
-		)
-		(property "Sheetfile" "motor_drive.kicad_sch"
-			(at 305.054 159.3346 0)
-			(effects
-				(font
-					(size 1.27 1.27)
-				)
-				(justify left top)
-			)
-		)
-		(instances
-			(project "skateboard"
-				(path "/5cdb5c16-5e05-458b-86f0-906cf8114d7e"
-					(page "6")
-				)
-			)
-		)
-	)
-	(sheet
-		(at 75.692 212.852)
-		(size 79.502 61.214)
-		(fields_autoplaced yes)
-		(stroke
-			(width 0.1524)
-			(type solid)
-		)
-		(fill
-			(color 0 0 0 0.0000)
-		)
-		(property "Sheetname" "ad转换"
-			(at 75.692 212.1404 0)
-			(effects
-				(font
-					(size 1.27 1.27)
-				)
-				(justify left bottom)
-			)
-		)
-		(property "Sheetfile" "ad_trans.kicad_sch"
-			(at 75.692 274.6506 0)
-			(effects
-				(font
-					(size 1.27 1.27)
-				)
-				(justify left top)
-			)
-		)
-		(instances
-			(project "skateboard"
-				(path "/5cdb5c16-5e05-458b-86f0-906cf8114d7e"
-					(page "4")
-				)
-			)
-		)
-	)
-	(sheet
-		(at 311.404 211.582)
-		(size 87.884 66.548)
-		(fields_autoplaced yes)
-		(stroke
-			(width 0.1524)
-			(type solid)
-		)
-		(fill
-			(color 0 0 0 0.0000)
-		)
-		(property "Sheetname" "GPS和音频"
-			(at 311.404 210.8704 0)
-			(effects
-				(font
-					(size 1.27 1.27)
-				)
-				(justify left bottom)
-			)
-		)
-		(property "Sheetfile" "GPS_Audio.kicad_sch"
-			(at 311.404 278.7146 0)
-			(effects
-				(font
-					(size 1.27 1.27)
-				)
-				(justify left top)
-			)
-		)
-		(instances
-			(project "skateboard"
-				(path "/5cdb5c16-5e05-458b-86f0-906cf8114d7e"
-					(page "7")
-				)
-			)
-		)
-	)
-	(sheet
-		(at 180.34 100.33)
-		(size 55.88 52.07)
-		(fields_autoplaced yes)
-		(stroke
-			(width 0.1524)
-			(type solid)
-		)
-		(fill
-			(color 0 0 0 0.0000)
-		)
-		(property "Sheetname" "dc-dc"
-			(at 180.34 99.6184 0)
-			(effects
-				(font
-					(size 1.27 1.27)
-				)
-				(justify left bottom)
-			)
-		)
-		(property "Sheetfile" "dc-dc.kicad_sch"
-			(at 180.34 152.9846 0)
-			(effects
-				(font
-					(size 1.27 1.27)
-				)
-				(justify left top)
-			)
-		)
-		(property "字段 2" ""
-			(at 180.34 100.33 0)
-			(effects
-				(font
-					(size 1.27 1.27)
-				)
-				(hide yes)
-			)
-		)
-		(instances
-			(project "skateboard"
-				(path "/5cdb5c16-5e05-458b-86f0-906cf8114d7e"
-					(page "2")
-				)
-			)
-		)
-	)
 	(sheet_instances
 		(path "/"
@@
 		)
 	)
+	(embedded_fonts no)
 )

Commit message: feat: update
Connections:
- no-connect marks 0 -> 4
Other:
- sheet 主控 renamed mcu
- added sheet foc1 (foc/foc.kicad_sch)
- added sheet foc2 (foc/foc.kicad_sch)
- sheet mcu: file main_ctrl.kicad_sch -> mcu.kicad_sch
- sheet mcu ports: added Battery_5V, IN1_1, IN1_2, IN1_3, IN2_1, IN2_2, IN2_3, MOT1_A, MOT1_B, MOT1_C, MOT2_A, MOT2_B, MOT2_C, current1_0, current1_1, current2_0, current2_1; removed none
- sheet power ports: added 3.3V/3A, 5V/3A; removed none

Commit message: feat: update
Parts:
- added J13, J14, J15, J16: Conn_01x01_Pin, MountingHole:MountingHole_4.3mm_M4, symbol Connector:Conn_01x01_Pin

Commit message: feat: update
Connections:
- no-connect marks 4 -> 8
Changed lines of the file:
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@@
 	(paper "A2")
 	(no_connect
+		(at 378.46 212.09)
+	)
+	(no_connect
 		(at 339.09 246.38)
+	)
+	(no_connect
+		(at 379.73 240.03)
+	)
+	(no_connect
+		(at 379.73 231.14)
 	)
 	(no_connect
@@
 	)
 	(no_connect
+		(at 378.46 222.25)
+	)
+	(no_connect
 		(at 339.09 237.49)
 	)
@@
 	(wire
 		(pts
+			(xy 264.16 203.2) (xy 264.16 213.36)
+		)
+		(stroke
+			(width 0)
+			(type default)
+		)
+	)
+	(wire
+		(pts
 			(xy 290.83 222.25) (xy 326.39 222.25)
 		)
@@
 	(wire
 		(pts
-			(xy 271.78 209.55) (xy 335.28 209.55)
+			(xy 273.05 209.55) (xy 335.28 209.55)
+		)
+		(stroke
+			(width 0)
+			(type default)
+		)
+	)
+	(wire
+		(pts
+			(xy 273.05 209.55) (xy 273.05 213.36)
 		)
 		(stroke
@@
 	(wire
 		(pts
-			(xy 264.16 203.2) (xy 264.16 213.36)
-		)
-		(stroke
-			(width 0)
-			(type default)
-		)
-	)
-	(wire
-		(pts
 			(xy 273.05 275.59) (xy 334.01 275.59)
 		)
@@
 		(pts
 			(xy 290.83 233.68) (xy 326.39 233.68)
-		)
-		(stroke
-			(width 0)
-			(type default)
-		)
-	)
-	(wire
-		(pts
-			(xy 271.78 213.36) (xy 271.78 209.55)
 		)
 		(stroke
@@
 		)
 		(pin "MOT1_C" input
-			(at 271.78 213.36 90)
+			(at 264.16 213.36 90)
 			(effects
 				(font
@@
 		)
 		(pin "MOT1_A" input
-			(at 264.16 213.36 90)
-			(effects
-				(font
+			(at 273.05 213.36 90)
+			(effects
+				(font
