File: pcb/mcu.kicad_sch (KiCad schematic)
At the start: 30 parts, among them J1 RC555, J2 pa1010d, J4 USB_C_Receptacle_USB2.0_16P, J5 UART, Q1 AO3401A, Q2 SS8050, Q3 SS8050, SW2 SW_Push, SW3 SW_Push, U3 ESP32-S3-WROOM-1

Commit message: feat: update
Parts:
- removed Q2, Q3: SS8050, Package_TO_SOT_SMD:SOT-23, symbol Transistor_BJT:SS8050
- removed R8: 10K, Resistor_SMD:R_0603_1608Metric, symbol CR0402JF0101G_2
- removed R9: 10K, Resistor_SMD:R_0603_1608Metric, symbol CR0402JF0101G_3
- J1: footprint Connector_PinHeader_2.54mm:PinHeader_1x08_P2.54mm_Vertical -> Connector_JST:JST_PH_B8B-PH-K_1x08_P2.00mm_Vertical
Connections:
- net DOUT_1: now also U3.32 (IO39); no longer U3.29 (IO36)
- net IN1_1: now also U3.30 (IO37); no longer U3.31 (IO38)
- net IN1_2: now also U3.29 (IO36); no longer U3.32 (IO39)
- net IN1_3: now also U3.28 (IO35); no longer U3.33 (IO40)
- net PD_SCK1: now also U3.33 (IO40); no longer U3.30 (IO37)
- net PD_SCK2: now also U3.31 (IO38); no longer U3.28 (IO35)
Other:
- note added: "Hall sensors"
- note added: "MOTOR PWMS"
- note added: "currents"
- note removed: "AUTO PROGRAM"
- note removed: "DTR RTS RST GPIO0 1 1 1 1 0 0 1 1 1 0 0 1 0 1 1 0"

Commit message: feat: update
Parts:
- removed RN2: 10k, Resistor_SMD:R_Array_Concave_4x0603, symbol Device:R_Pack04
- added R58, R59, R8, R9: 10K, Resistor_SMD:R_0603_1608Metric, symbol Device:R
- D10: value LED -> TXD
- D7: value 3.3v -> +3.3v
- D9: value LED -> RXD
- SW2: value SW_Push -> BOOT
- SW3: value SW_Push -> EN
Connections:
- net +3.3V: now also R9.1
- net IN1_1: now also U3.19 (IO11); no longer U3.30 (IO37)
- net IN1_2: now also U3.18 (IO10); no longer U3.29 (IO36)
- net IN1_3: now also U3.17 (IO9); no longer U3.28 (IO35)
- net IN2_1: now also U3.22 (IO14); no longer U3.34 (IO41)
- net IN2_2: now also U3.21 (IO13); no longer U3.35 (IO42)
- net IN2_3: now also U3.20 (IO12); no longer U3.26 (IO45)
- net MOT1_A: now also U3.26 (IO45); no longer U3.17 (IO9)
- net MOT1_B: now also U3.35 (IO42); no longer U3.18 (IO10)
- net MOT1_C: now also U3.34 (IO41); no longer U3.19 (IO11)
- net MOT2_A: now also U3.30 (IO37); no longer U3.20 (IO12)
- net MOT2_B: now also U3.29 (IO36); no longer U3.21 (IO13)
- net MOT2_C: now also U3.28 (IO35); no longer U3.22 (IO14)
- net U0_RXD: now also R58.1
- net U0_TXD: now also R59.1
- net VBUS: now also R8.1
- net at D6.2 (A): now also R8.2
- net at D7.2 (A): now also R9.2
- net at D9.1 (K): now also R58.2
- net at D10.1 (K): now also R59.2
Other:
- moved on the sheet: D1, D2, D3

Commit message: feat: update
Connections:
- net DOUT_1: now also U3.9 (IO16); no longer U3.32 (IO39)
- net DOUT_2: now also U3.24 (IO47); no longer U3.23 (IO21)
- net IRQ: now also U3.39 (IO1); no longer U3.38 (IO2)
- net MOSI: now also U3.12 (IO8); no longer U3.4 (IO4)
- net MOT1_A: now also U3.31 (IO38); no longer U3.26 (IO45)
- net MOT1_B: now also U3.34 (IO41); no longer U3.35 (IO42)
- net MOT1_C: now also U3.35 (IO42); no longer U3.34 (IO41)
- net PD_SCK1: now also U3.8 (IO15); no longer U3.33 (IO40)
- net PD_SCK2: now also U3.23 (IO21); no longer U3.31 (IO38)
- net RST: now also U3.38 (IO2); no longer U3.39 (IO1)
- net SCK: now also U3.33 (IO40); no longer U3.8 (IO15)
- net SDA: now also U3.32 (IO39); no longer U3.9 (IO16)
- net current1_1: now also U3.4 (IO4); no longer U3.6 (IO6)
- net current2_0: now also U3.6 (IO6); no longer U3.7 (IO7)
- net current2_1: now also U3.7 (IO7); no longer U3.12 (IO8)
- net MOTO_POWER: now reaches U3.16 (IO46)
- no-connect marks 6 -> 5

Commit message: update
Parts:
- D4, D5: value MBR120VLSFT1G -> B560C
Changed lines of the file:
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@@
 (kicad_sch
-	(version 20250227)
+	(version 20250318)
 	(generator "eeschema")
 	(generator_version "9.99")
@@
 			)
 		)
-		(property "Datasheet" "~"
+		(property "Datasheet" ""
 			(at 121.92 44.45 0)
 			(hide yes)
@@
 			)
 		)
-		(property "Datasheet" "~"
+		(property "Datasheet" ""
 			(at 78.74 35.56 0)
 			(hide yes)
@@
 			)
 		)
-		(property "Datasheet" "~"
+		(property "Datasheet" ""
 			(at 113.03 175.26 0)
 			(hide yes)
@@
 			)
 		)
-		(property "Value" "MBR120VLSFT1G"
+		(property "Value" "B560C"
 			(at 214.122 117.602 0)
 			(effects
@@
 			)
 		)
-		(property "Datasheet" "~"
+		(property "Datasheet" ""
 			(at 208.28 120.65 0)
 			(hide yes)
@@
 			)
 		)
-		(property "Datasheet" "~"
+		(property "Datasheet" ""
 			(at 85.09 171.45 0)
 			(hide yes)
@@
 			)
 		)
-		(property "Datasheet" "~"
+		(property "Datasheet" ""
 			(at 185.42 144.78 0)
 			(hide yes)
@@
 			)
 		)
-		(property "Datasheet" "~"
+		(property "Datasheet" ""
 			(at 245.11 138.43 0)
 			(hide yes)
@@
 			)
 		)
-		(property "Datasheet" "~"
+		(property "Datasheet" ""
 			(at 76.2 44.45 0)
 			(hide yes)
@@
 			)
 		)
-		(property "Datasheet" "~"
+		(property "Datasheet" ""
 			(at 121.92 58.42 0)
 			(hide yes)
@@
 			)
 		)
-		(property "Datasheet" "~"
+		(property "Datasheet" ""
 			(at 252.73 121.92 0)
 			(hide yes)
@@
 			)
 		)
-		(property "Datasheet" "~"
+		(property "Datasheet" ""
 			(at 167.64 68.58 0)
 			(hide yes)
@@
 			)
 		)
-		(property "Datasheet" "~"
+		(property "Datasheet" ""
 			(at 76.2 46.99 0)
 			(hide yes)
@@
 			)
 		)
-		(property "Datasheet" "~"
+		(property "Datasheet" ""
 			(at 250.19 121.92 0)
 			(hide yes)
@@
 			)
 		)
-		(property "Datasheet" "~"
+		(property "Datasheet" ""
 			(at 237.49 138.43 0)
 			(hide yes)
@@
 			)
 		)
-		(property "Datasheet" "~"
+		(property "Datasheet" ""
 			(at 255.27 121.92 0)
 			(hide yes)
@@
 			)
 		)
-		(property "Datasheet" "~"
+		(property "Datasheet" ""
 			(at 167.64 39.37 0)
 			(hide yes)
@@
 			)
 		)
-		(property "Datasheet" "~"
+		(property "Datasheet" ""
 			(at 153.67 39.37 0)
 			(hide yes)
@@
 			)
 		)
-		(property "Datasheet" "~"
+		(property "Datasheet" ""
 			(at 153.67 67.31 0)
 			(hide yes)
@@
 			)
 		)
-		(property "Datasheet" "~"
+		(property "Datasheet" ""
 			(at 137.16 175.26 0)
 			(hide yes)
@@
 			)
 		)
-		(property "Datasheet" "~"
+		(property "Datasheet" ""
 			(at 247.65 121.92 0)
 			(hide yes)
@@
 			)
 		)
-		(property "Datasheet" "~"
+		(property "Datasheet" ""
 			(at 265.43 138.43 0)
 			(hide yes)
@@
 			)
 		)
-		(property "Datasheet" "~"
+		(property "Datasheet" ""
 			(at 257.81 138.43 0)
 			(hide yes)
@@
 			)
 		)
-		(property "Value" "MBR120VLSFT1G"
+		(property "Value" "B560C"
 			(at 192.532 113.284 0)
 			(effects
@@
 			)
 		)
-		(property "Datasheet" "~"
+		(property "Datasheet" ""
 			(at 195.58 120.65 0)
 			(hide yes)

Commit message: update
Parts:
- added J17: Conn_01x02_Pin, Connector_PinSocket_2.54mm:PinSocket_1x02_P2.54mm_Vertical, symbol Connector:Conn_01x02_Pin
Connections:
- net DOUT_2: now also U3.23 (IO21); no longer U3.24 (IO47)
- net PD_SCK2: now also U3.24 (IO47); no longer U3.23 (IO21)
- net Battery_RXD: now reaches U3.25 (IO48)
- net Battery_RXD: now also J17.2 (Pin_2)
- net Battery_TXD: now reaches U3.26 (IO45)
- net Battery_TXD: now also J17.1 (Pin_1)
- no-connect marks 5 -> 3
Changed lines of the file:
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@@
 		(at 72.39 67.31)
 	)
-	(no_connect
-		(at 78.74 148.59)
-	)
-	(no_connect
-		(at 78.74 156.21)
-	)
 	(wire
 		(pts
@@
 		)
 	)
+	(global_label "PD_SCK2"
+		(shape input)
+		(at 78.74 153.67 0)
+		(fields_autoplaced yes)
+		(effects
+			(font
+				(size 1.27 1.27)
+			)
+			(justify left)
+		)
+		(property "Intersheetrefs" "${INTERSHEET_REFS}"
+			(at 90.1918 153.67 0)
+			(hide yes)
+			(effects
+				(font
+					(size 1.27 1.27)
+				)
+				(justify left)
+			)
+		)
+	)
 	(global_label "EN"
 		(shape input)
@@
 		)
 	)
+	(global_label "Battery_TXD"
+		(shape input)
+		(at 121.92 147.32 0)
+		(fields_autoplaced yes)
+		(effects
+			(font
+				(size 1.27 1.27)
+			)
+			(justify left)
+		)
+		(property "Intersheetrefs" "${INTERSHEET_REFS}"
+			(at 136.0327 147.32 0)
+			(hide yes)
+			(effects
+				(font
+					(size 1.27 1.27)
+				)
+				(justify left)
+			)
+		)
+	)
+	(global_label "DOUT_2"
+		(shape input)
+		(at 78.74 125.73 0)
+		(fields_autoplaced yes)
+		(effects
+			(font
+				(size 1.27 1.27)
+			)
+			(justify left)
+		)
+		(property "Intersheetrefs" "${INTERSHEET_REFS}"
+			(at 88.8009 125.73 0)
+			(hide yes)
+			(effects
+				(font
+					(size 1.27 1.27)
+				)
+				(justify left)
+			)
+		)
+	)
 	(global_label "TXD_SENSOR"
 		(shape input)
@@
 		)
 	)
-	(global_label "DOUT_2"
-		(shape input)
-		(at 78.74 153.67 0)
-		(fields_autoplaced yes)
-		(effects
-			(font
-				(size 1.27 1.27)
-			)
-			(justify left)
-		)
-		(property "Intersheetrefs" "${INTERSHEET_REFS}"
-			(at 88.8009 153.67 0)
-			(hide yes)
-			(effects
-				(font
-					(size 1.27 1.27)
-				)
-				(justify left)
-			)
-		)
-	)
 	(global_label "SDA"
 		(shape input)
@@
 		)
 	)
-	(global_label "PD_SCK2"
-		(shape input)
-		(at 78.74 125.73 0)
-		(fields_autoplaced yes)
-		(effects
-			(font
-				(size 1.27 1.27)
-			)
-			(justify left)
-		)
-		(property "Intersheetrefs" "${INTERSHEET_REFS}"
-			(at 90.1918 125.73 0)
-			(hide yes)
-			(effects
-				(font
-					(size 1.27 1.27)
-				)
-				(justify left)
-			)
-		)
-	)
 	(global_label "U0_RXD"
 		(shape input)
@@
 		)
 	)
+	(global_label "Battery_RXD"
+		(shape input)
+		(at 121.92 149.86 0)
+		(fields_autoplaced yes)
+		(effects
+			(font
+				(size 1.27 1.27)
+			)
+			(justify left)
+		)
+		(property "Intersheetrefs" "${INTERSHEET_REFS}"
+			(at 136.3351 149.86 0)
+			(hide yes)
+			(effects
+				(font
+					(size 1.27 1.27)
+				)
+				(justify left)
+			)
+		)
+	)
 	(global_label "USB_D-"
 		(shape input)
@@
 					(size 1.27 1.27)
 				)
+			)
+		)
+	)
+	(global_label "Battery_TXD"
+		(shape input)
+		(at 78.74 148.59 0)
+		(fields_autoplaced yes)
+		(effects
+			(font
+				(size 1.27 1.27)
+			)
+			(justify left)
+		)
+		(property "Intersheetrefs" "${INTERSHEET_REFS}"
+			(at 92.8527 148.59 0)
+			(hide yes)
+			(effects
+				(font
+					(size 1.27 1.27)
+				)
+				(justify left)
 			)
 		)
@@
 				)
 				(justify right)
+			)
+		)
+	)
+	(global_label "Battery_RXD"
+		(shape input)
+		(at 78.74 156.21 0)
+		(fields_autoplaced yes)
+		(effects
+			(font
+				(size 1.27 1.27)
+			)
+			(justify left)
+		)
+		(property "Intersheetrefs" "${INTERSHEET_REFS}"
+			(at 93.1551 156.21 0)
+			(hide yes)
+			(effects
+				(font
+					(size 1.27 1.27)
+				)
+				(justify left)
 			)
 		)
@@
 					(unit 1)
 				)
+			)
+		)
+	)
+	(symbol
+		(lib_id "Connector:Conn_01x02_Pin")
+		(at 116.84 147.32 0)
+		(unit 1)
+		(exclude_from_sim no)
+		(in_bom yes)
+		(on_board yes)
+		(dnp no)
+		(fields_autoplaced yes)
+		(property "Reference" "J17"
+			(at 117.475 142.24 0)
+			(effects
+				(font
+					(size 1.27 1.27)
+				)
+			)
+		)
+		(property "Value" "Conn_01x02_Pin"
+			(at 117.475 144.78 0)
+			(effects
+				(font
+					(size 1.27 1.27)
+				)
+			)
+		)
+		(property "Footprint" "Connector_PinSocket_2.54mm:PinSocket_1x02_P2.54mm_Vertical"
+			(at 116.84 147.32 0)
+			(hide yes)
+			(effects
+				(font
+					(size 1.27 1.27)
+				)
+			)
+		)
+		(property "Datasheet" ""
+			(at 116.84 147.32 0)
+			(hide yes)
+			(effects
+				(font
+					(size 1.27 1.27)
+				)
+			)
+		)
+		(property "Description" "Generic connector, single row, 01x02, script generated"
+			(at 116.84 147.32 0)
+			(hide yes)
+			(effects
+				(font
+					(size 1.27 1.27)
+				)
+			)
+		)
+		(pin "2"
+		)
+		(pin "1"
+		)
+		(instances
+			(project ""
+				(path "/5cdb5c16-5e05-458b-86f0-906cf8114d7e/5f743cab-9820-4aca-8ca5-f45b69affbe2"
+					(reference "J17")
+					(unit 1)
+				)
