File: pcb/sensor/sensor.kicad_pcb (KiCad board)
At the start: 2 copper layers, 25.5 x 23 mm, 15 parts, among them J3 sig_in, J4 sig_out, J5 Conn_01x02_Pin, J6 Conn_01x02_Pin, J7 Conn_02x02_Counter_Clockwise, U1 TJA1051T-3, U2 HX711

Commit message: feat: update dc-dc
Parts:
- added C12: 100nF, Capacitor_SMD:C_0603_1608Metric, F.Cu at (167.2, 51.5)
- added C13: 100nF, Capacitor_SMD:C_0603_1608Metric, F.Cu at (167.2, 54.0)
- added C7: 100nF, Capacitor_SMD:C_0603_1608Metric, F.Cu at (167.2, 49.0)
- added R1: 100k, Resistor_SMD:R_0603_1608Metric, F.Cu at (167.2, 56.5)
- added R4: 6.67k, Resistor_SMD:R_0603_1608Metric, F.Cu at (167.2, 59.0)
- added R7: 50K, Resistor_SMD:R_0603_1608Metric, F.Cu at (167.2, 61.5)
- added U3: LM2595S-3.3, Package_TO_SOT_SMD:TO-263-5_TabPin3, F.Cu at (158.2, 53.9)
- added U4: LM2595S-5, Package_TO_SOT_SMD:TO-263-5_TabPin3, F.Cu at (158.2, 66.2)

Commit message: feat: update
Parts:
- removed C12, C2, C7: 100nF, Capacitor_SMD:C_0603_1608Metric
- removed C5: 1uF, Capacitor_SMD:C_0603_1608Metric
- removed J5, J6: Conn_01x02_Pin, Connector_PinHeader_2.54mm:PinHeader_1x02_P2.54mm_Vertical
- removed R5, R6: 60, Resistor_SMD:R_0603_1608Metric
- removed U3: LM2595S-3.3, Package_TO_SOT_SMD:TO-263-5_TabPin3
- removed U4: LM2595S-5, Package_TO_SOT_SMD:TO-263-5_TabPin3
- added C14: 68nF, Capacitor_SMD:C_0603_1608Metric, F.Cu at (132.8, 62.9)
- added C15: 10uF/35v, Capacitor_SMD:C_1210_3225Metric, F.Cu at (144.5, 76.3)
- added C17: 10uF/35v, Capacitor_SMD:C_1210_3225Metric, F.Cu at (144.5, 80.6)
- added C18: 10uf/50v, Capacitor_SMD:C_1210_3225Metric, F.Cu at (144.5, 84.8)
- added C19: 10uf/50v, Capacitor_SMD:C_1210_3225Metric, F.Cu at (144.5, 89.1)
- added C20: 100nf/50v, Capacitor_SMD:C_0603_1608Metric, F.Cu at (132.8, 65.4)
- added C21: 4.7uf/50v, Capacitor_SMD:C_1206_3216Metric, F.Cu at (158.2, 55.8)
- added C22: 100nf/50v, Capacitor_SMD:C_0603_1608Metric, F.Cu at (132.8, 68.0)
- added C24: 47nF, Capacitor_SMD:C_0603_1608Metric, F.Cu at (132.8, 70.5)
- added C25: 100nF/16v, Capacitor_SMD:C_0603_1608Metric, F.Cu at (132.8, 73.0)
- added C26: 10uF/10v, Capacitor_SMD:C_0603_1608Metric, F.Cu at (136.8, 55.4)
- added C27: 10uF/10v, Capacitor_SMD:C_0603_1608Metric, F.Cu at (136.8, 57.9)
- added C28: 4.7uf/50v, Capacitor_SMD:C_1206_3216Metric, F.Cu at (158.2, 59.2)
- added C30: 4.7uf/50v, Capacitor_SMD:C_1206_3216Metric, F.Cu at (158.2, 62.5)
- added C31: 47nF, Capacitor_SMD:C_0603_1608Metric, F.Cu at (136.8, 60.4)
- added C32: 100nF/16v, Capacitor_SMD:C_0603_1608Metric, F.Cu at (136.8, 62.9)
- added C33: 10uF/16v, Capacitor_SMD:C_1210_3225Metric, F.Cu at (144.5, 93.3)
- added C34: 10uF/16v, Capacitor_SMD:C_1210_3225Metric, F.Cu at (144.5, 97.6)
- added D3: B560C, Diode_SMD:D_SMC, F.Cu at (136.3, 78.1)
- added D6: B560C, Diode_SMD:D_SMC, F.Cu at (136.3, 85.8)
- added D7: B560C, Diode_SMD:D_SMC, F.Cu at (136.3, 93.6)
- added L3: 22uH, Inductor_SMD:L_TDK_SLF12565, F.Cu at (123.2, 61.5)
- added L4: 22uH, Inductor_SMD:L_TDK_SLF12565, F.Cu at (123.2, 75.8)
- added L5: 47uH, Inductor_SMD:L_TDK_SLF12565, F.Cu at (123.2, 90.1)
- added R10: 10k, Resistor_SMD:R_0603_1608Metric, F.Cu at (140.8, 57.9)
- added R11: 62k, Resistor_SMD:R_0603_1608Metric, F.Cu at (140.8, 60.4)
- added R12: 33k, Resistor_SMD:R_0603_1608Metric, F.Cu at (140.8, 62.9)
- added R13: 1k, Resistor_SMD:R_0603_1608Metric, F.Cu at (140.8, 65.4)
- added R14: 10k, Resistor_SMD:R_0603_1608Metric, F.Cu at (140.8, 68.0)
- added R15: 62k, Resistor_SMD:R_0603_1608Metric, F.Cu at (140.8, 70.5)
- added R16: 56k, Resistor_SMD:R_0603_1608Metric, F.Cu at (140.8, 73.0)
- added R17: 680, Resistor_SMD:R_0603_1608Metric, F.Cu at (144.8, 55.4)
- added R18: 10k, Resistor_SMD:R_0603_1608Metric, F.Cu at (144.8, 57.9)
- added R19: 1.3k, Resistor_SMD:R_0603_1608Metric, F.Cu at (144.8, 60.4)
- added R20: 1.3k, Resistor_SMD:R_0603_1608Metric, F.Cu at (144.8, 62.9)
- added R21: 120, Resistor_SMD:R_0603_1608Metric, F.Cu at (144.8, 65.4)
- added SW2: SW_SPST, Button_Switch_SMD:SW_DIP_SPSTx01_Slide_Copal_CHS-01A_W5.08mm_P1.27mm_JPin, F.Cu at (119.7, 99.2)
- added U5: LMR16030SDDAR, Package_SO:TI_SO-PowerPAD-8_ThermalVias, F.Cu at (151.6, 77.6)
- added U8: LMR16030SDDAR, Package_SO:TI_SO-PowerPAD-8_ThermalVias, F.Cu at (151.6, 84.3)
- added U9: LMR16030SDDAR, Package_SO:TI_SO-PowerPAD-8_ThermalVias, F.Cu at (151.6, 90.9)
- C13: value 100nF -> 100nF/16v
- R1: value 100k -> 300k
- R4: value 6.67k -> 10k
- R7: value 50K -> 100k
- U1: value TJA1051T-3 -> SIT1042AQT/3; footprint Package_SO:SOIC-8_3.9x4.9mm_P1.27mm -> Package_DFN_QFN:DFN-8-1EP_3x3mm_P0.65mm_EP1.5x2.25mm
- moved C13 35.0 mm to (132.8, 60.4)
- moved C3 33.9 mm to (132.8, 55.4), turned to 0 degrees
- moved R4 33.4 mm to (136.8, 73.0)
- moved U2 32.7 mm to (151.1, 60.0)
- moved R1 31.7 mm to (136.8, 65.4)
- moved J3 29.3 mm to (149.2, 68.1)
- moved R7 27.0 mm to (140.8, 55.4)
- moved R2 26.0 mm to (136.8, 68.0), turned to 0 degrees
- moved U1 24.5 mm to (157.6, 96.5), turned to 0 degrees
- moved C6 23.1 mm to (132.8, 57.9), turned to 0 degrees
- moved R3 22.6 mm to (136.8, 70.5), turned to 0 degrees
- moved J4 20.6 mm to (153.8, 68.1), turned to 0 degrees
- moved J7 16.3 mm to (149.7, 96.5)
Connections:
- net 12V/3A renamed 24V/3A
- R1 pad 2: Net-(U5-FB) -> Net-(R1-Pad2)
- U1 pad 8: STANDBY -> GND
Routing:
- net +5V: track 43.0 -> 0.00 mm
- net +3.3V: track 33.3 -> 0.00 mm
- net CANH: track 11.6 -> 0.00 mm
- net GND: track 10.6 -> 0.00 mm, vias 3 -> 0
- net PD_SCK: track 10.5 -> 0.00 mm
- net CANL: track 9.92 -> 0.00 mm
- net DOUT: track 7.48 -> 0.00 mm
- net INA-: track 7.30 -> 0.00 mm
- net INA+: track 6.56 -> 0.00 mm
- net RXD: track 5.74 -> 0.00 mm
- net TXD: track 5.69 -> 0.00 mm
- net Net-(U2-INA-): track 4.59 -> 0.00 mm
- net Net-(U2-INA+): track 4.48 -> 0.00 mm
- net Net-(C5-Pad2): track 3.42 -> 0.00 mm
- removed copper zone on B.Cu, net GND
- removed copper zone on F.Cu, net GND
Other:
- board outline removed
