File: pcb/foc/foc.kicad_sch (KiCad schematic)
At the start: 44 parts, among them J6 TB_MOTOR, J7 PH_2.0, Q4 BTN8982TA, Q5 BTN8982TA, Q6 BTN8982TA, U7 INA240A2PW, U8 INA240A2PW

Commit message: feat: update
Parts:
- removed 3.3V2, 42V2: LED, LED_SMD:LED_0603_1608Metric, symbol Device:LED
- removed C28, C29: 330uf, Capacitor_SMD:CP_Elec_10x10.5, symbol Device:C_Polarized
- removed C37: 100nF, Capacitor_SMD:C_0603_1608Metric, symbol Device:C
- removed C39: 20pF, Capacitor_SMD:C_0603_1608Metric, symbol Device:C
- removed R37: 1k, Resistor_SMD:R_0603_1608Metric, symbol Device:R_US
- removed R43: 3.3k, Resistor_SMD:R_0603_1608Metric, symbol Device:R_US
- added C53: 20pF, Capacitor_SMD:C_0603_1608Metric, symbol Device:C
- added C54: 100nF, Capacitor_SMD:C_0603_1608Metric, symbol Device:C
- C34: value 100nF -> 20pF
- C35: value 20pF -> 100nF
- R35: value 10k -> 3.3k
Connections:
- net +3.3V: now also R35.2, R38.2; no longer R38.1
- net GND: now also C34.1, C35.2, C53.1, C54.2; no longer C34.2, C35.1
- net MOT_A: now also C30.1, C31.2, R33.1; no longer C34.1, C35.2, R38.2
- net MOT_B: now also C34.2, C35.1, R35.1
- net MOT_C: now also R38.1, C53.2, C54.1; no longer C30.1, C31.2, R33.1
- net VCC: no longer R35.1
Other:
- moved on the sheet: C30, C31, J6, J7, R33

Commit message: feat: update
Parts:
- C40, C41: value 0.1nF -> 0.1uF
Connections:
- net GND: now also C40.1, C41.1, U7.7 (REF1), U8.7 (REF1)
- net out1: no longer names the net of J6.1 (Pin_1), R44.1, U7.2 (+)
- net out1_cs: no longer names the net of Q4.4, Q4.8, R44.2, U7.3 (-)
- net out2: no longer names the net of J6.2 (Pin_2), Q5.4, Q5.8
- net out3: no longer names the net of J6.3 (Pin_3), R45.2, U8.3 (-)
- net out3_cs: no longer names the net of Q6.4, Q6.8, R45.1, U8.2 (+)
Other:
- moved on the sheet: C26, C27, C30, C31, C32, C33, C34, C35, C36, C38, C40, C41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

Commit message: feat: update
Parts:
- C40, C41: value 0.1uF -> 100nF
Connections:
- net +3.3V: no longer R27.2, R31.2, R39.2
- new net MOTO_POWER: R27.2, R31.2, R39.2
Other:
- note added: "High enable"
- moved on the sheet: U8

Commit message: update
Parts:
- added C24, C6: 100nf, Capacitor_SMD:C_0603_1608Metric, symbol Device:C
- added R64, R68: 200k, Resistor_SMD:R_0603_1608Metric, symbol Device:R
Connections:
- net +3.3V: now also R64.2, R68.2; no longer U7.6 (REF2), U8.6 (REF2)
- net A0: now also C6.1
- net A1: now also C24.1
- net GND: now also C24.2, C6.2
- net at J6.1 (Pin_1), R44.1: now also U7.3 (-); no longer U7.2 (+)
- net at Q4.4, Q4.8, R44.2: now also U7.2 (+); no longer U7.3 (-)
- net at J6.3 (Pin_3), R45.2: now also U8.2 (+); no longer U8.3 (-)
- net at Q6.4, Q6.8, R45.1: now also U8.3 (-); no longer U8.2 (+)
- new net: R64.1, U8.6 (REF2)
- new net: R68.1, U7.6 (REF2)
Other:
- moved on the sheet: C40, C41
