File: pcb/battery/battery.kicad_sch (KiCad schematic)
At the start: 75 parts, among them J1 Conn_01x11_Pin, J2 p2.0, J3 p2.0, J4 UART XH2.54, J5 p2.0, J6 P+/C+, J7 PN/CN, J8 B+, J9 B-, Q1 MMBT5401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

Commit message: feat: update
Parts:
- removed J2, J3, J5: p2.0, Connector_PinHeader_2.00mm:PinHeader_1x02_P2.00mm_Vertical, symbol Connector:Conn_01x02_Pin
- removed NT1: power, NetTie:NetTie-2_SMD_Pad0.5mm, symbol Device:NetTie_2
- removed NT3: sensor, NetTie:NetTie-2_SMD_Pad0.5mm, symbol Device:NetTie_2
- added J10: Conn_01x06_Pin, Connector_JST:JST_PH_B6B-PH-K_1x06_P2.00mm_Vertical, symbol Connector:Conn_01x06_Pin
- J6, J7: footprint MountingHole:MountingHole_4.3mm_M4_DIN965_Pad -> MountingHole:MountingHole_2.2mm_M2_DIN965_Pad_TopBottom
- J8: value B+ -> PN/CN; footprint MountingHole:MountingHole_4.3mm_M4_DIN965_Pad -> MountingHole:MountingHole_2.2mm_M2_DIN965_Pad_TopBottom
- J9: value B- -> P+/C+; footprint MountingHole:MountingHole_4.3mm_M4_DIN965_Pad -> MountingHole:MountingHole_2.2mm_M2_DIN965_Pad_TopBottom
Connections:
- net B+/P+/C+: now also J9.1 (Pin_1); no longer J8.1 (Pin_1)
- net GND: now also C2.1, J8.1 (Pin_1), R10.1, R11.2, R12.2, R13.2, R14.2, R2.1, J10.2 (Pin_2), J10.4 (Pin_4), J10.6 (Pin_6)
- net at C21.1, U1.18 (TS3): now also J10.5 (Pin_5)
- net at C20.1, U1.17 (TS2): now also J10.3 (Pin_3)
- net at C17.1, U1.16 (TS1): now also J10.1 (Pin_1)
- removed net B-: C2.1, J9.1 (Pin_1), R10.1, R11.2, R12.2, R13.2, R14.2, R2.1
Other:
- moved on the sheet: C17, C20, C21
