File: pcb/dc-dc/dc-dc.kicad_sch (KiCad schematic)
At the start: 50 parts, among them J8 power, U4 LMR16030SDDAR, U5 LMR16030SDDAR, U6 LMR16030SDDAR

Commit message: feat: update
Parts:
- C12, C13, C19: value 100nF/16v -> 100nF
- C8: value 100nf/50v -> 100nf
Changed lines of the file:
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@@
 			)
 		)
-		(property "Value" "100nF/16v"
+		(property "Value" "100nF"
 			(at 118.11 36.83 90)
 			(effects
@@
 			)
 		)
-		(property "Value" "100nF/16v"
+		(property "Value" "100nF"
 			(at 182.88 100.33 90)
 			(effects
@@
 			)
 		)
-		(property "Value" "100nf/50v"
+		(property "Value" "100nf"
 			(at 53.594 47.752 0)
 			(effects
@@
 			)
 		)
-		(property "Value" "100nF/16v"
+		(property "Value" "100nF"
 			(at 245.11 39.37 90)
 			(effects

Commit message: feat: udpate pcb
Parts:
- L2: value 22uH -> 10uH
Changed lines of the file:
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@@
 			)
 		)
-		(property "Value" "22uH"
+		(property "Value" "10uH"
 			(at 242.824 53.594 90)
 			(effects
